File: hardware/antenna_block.sch (KiCad schematic (older format))
At the start: 27 parts, among them P301 BNC

Commit message: Linked first components to footprints and updated schematic plot
Parts:
- C301, C302, C303, C304, C305, C306, C307, C308, C309, C310, C311: footprint (none) -> Capacitors_SMD:C_0805
- D301, D302, D303: value BAT83 -> BAT54; footprint (none) -> TO_SOT_Packages_SMD:SOT-23_Handsoldering
- R301, R302, R303, R304, R305: footprint (none) -> Resistors_SMD:R_0805_HandSoldering
Changed lines of the file:
@@
 F 0 "P301" H 2810 3220 50  0000 C CNN
 F 1 "BNC" V 2910 3040 50  0000 C CNN
-F 2 "" H 2800 3100 50  0000 C CNN
+F 2 "" H 2800 3100 50  0001 C CNN
 F 3 "" H 2800 3100 50  0000 C CNN
 	1    2800 3100
@@
 F 0 "C301" H 3160 3170 50  0000 L CNN
 F 1 "1nF" H 3160 3020 50  0000 L CNN
-F 2 "" H 3150 3100 50  0000 C CNN
+F 2 "Capacitors_SMD:C_0805" H 3150 3100 50  0001 C CNN
 F 3 "" H 3150 3100 50  0000 C CNN
 	1    3150 3100
@@
 F 0 "C302" H 3410 3370 50  0000 L CNN
 F 1 "1nF" H 3410 3220 50  0000 L CNN
-F 2 "" H 3400 3300 50  0000 C CNN
+F 2 "Capacitors_SMD:C_0805" H 3400 3300 50  0001 C CNN
 F 3 "" H 3400 3300 50  0000 C CNN
 	1    3400 3300
@@
 $EndComp
 $Comp
-L GND #PWR301
+L GND #PWR013
 U 1 1 57E329F5
 P 3800 3550
-F 0 "#PWR301" H 3800 3300 50  0001 C CNN
+F 0 "#PWR013" H 3800 3300 50  0001 C CNN
 F 1 "GND" H 3800 3400 50  0000 C CNN
 F 2 "" H 3800 3550 50  0000 C CNN
@@
 F 0 "L301" H 3630 3140 50  0000 L CNN
 F 1 "660nH" H 3630 3060 50  0000 L CNN
-F 2 "" H 3600 3100 50  0000 C CNN
+F 2 "" H 3600 3100 50  0001 C CNN
 F 3 "" H 3600 3100 50  0000 C CNN
 	1    3600 3100
@@
 F 0 "L302" H 4030 3140 50  0000 L CNN
 F 1 "660nH" H 4030 3060 50  0000 L CNN
-F 2 "" H 4000 3100 50  0000 C CNN
+F 2 "" H 4000 3100 50  0001 C CNN
 F 3 "" H 4000 3100 50  0000 C CNN
 	1    4000 3100
@@
 F 0 "C303" H 3810 3370 50  0000 L CNN
 F 1 "3nF" H 3810 3220 50  0000 L CNN
-F 2 "" H 3800 3300 50  0000 C CNN
+F 2 "Capacitors_SMD:C_0805" H 3800 3300 50  0001 C CNN
 F 3 "" H 3800 3300 50  0000 C CNN
 	1    3800 3300
@@
 F 0 "C304" H 4210 3370 50  0000 L CNN
 F 1 "1nF" H 4210 3220 50  0000 L CNN
-F 2 "" H 4200 3300 50  0000 C CNN
+F 2 "Capacitors_SMD:C_0805" H 4200 3300 50  0001 C CNN
 F 3 "" H 4200 3300 50  0000 C CNN
 	1    4200 3300
@@
 F 0 "C305" H 4460 3170 50  0000 L CNN
 F 1 "1nF" H 4460 3020 50  0000 L CNN
-F 2 "" H 4450 3100 50  0000 C CNN
+F 2 "Capacitors_SMD:C_0805" H 4450 3100 50  0001 C CNN
 F 3 "" H 4450 3100 50  0000 C CNN
 	1    4450 3100
@@
 F 0 "R302" H 4680 3570 50  0000 L CNN
 F 1 "50R" H 4680 3510 50  0000 L CNN
-F 2 "" H 4650 3550 50  0000 C CNN
+F 2 "Resistors_SMD:R_0805_HandSoldering" H 4650 3550 50  0001 C CNN
 F 3 "" H 4650 3550 50  0000 C CNN
 	1    4650 3550
@@
 F 0 "R303" H 5680 3570 50  0000 L CNN
 F 1 "50R" H 5680 3510 50  0000 L CNN
-F 2 "" H 5650 3550 50  0000 C CNN
+F 2 "Resistors_SMD:R_0805_HandSoldering" H 5650 3550 50  0001 C CNN
 F 3 "" H 5650 3550 50  0000 C CNN
 	1    5650 3550
@@
 F 0 "R301" H 4330 3920 50  0000 L CNN
 F 1 "10k" H 4330 3860 50  0000 L CNN
-F 2 "" H 4300 3900 50  0000 C CNN
+F 2 "Resistors_SMD:R_0805_HandSoldering" H 4300 3900 50  0001 C CNN
 F 3 "" H 4300 3900 50  0000 C CNN
 	1    4300 3900
@@
 U 1 1 57E32A3A
 P 4400 4200
-F 0 "D301" H 4350 4280 50  0000 L CNN
-F 1 "BAT83" H 4120 4120 50  0000 L CNN
-F 2 "" V 4400 4200 50  0000 C CNN
+F 0 "D301" H 4250 4300 50  0000 L CNN
+F 1 "BAT54" H 4300 4100 50  0000 L CNN
+F 2 "TO_SOT_Packages_SMD:SOT-23_Handsoldering" V 4400 4200 50  0001 C CNN
 F 3 "" V 4400 4200 50  0000 C CNN
 	1    4400 4200
@@
 U 1 1 57E32A41
 P 4950 3550
-F 0 "D302" H 4900 3630 50  0000 L CNN
-F 1 "BAT83" H 4670 3470 50  0000 L CNN
-F 2 "" V 4950 3550 50  0000 C CNN
+F 0 "D302" H 4700 3600 50  0000 L CNN
+F 1 "BAT54" H 4850 3450 50  0000 L CNN
+F 2 "TO_SOT_Packages_SMD:SOT-23_Handsoldering" V 4950 3550 50  0001 C CNN
 F 3 "" V 4950 3550 50  0000 C CNN
 	1    4950 3550
@@
 P 5350 3550
 F 0 "D303" H 5300 3630 50  0000 L CNN
-F 1 "BAT83" H 5070 3470 50  0000 L CNN
-F 2 "" V 5350 3550 50  0000 C CNN
+F 1 "BAT54" H 5200 3450 50  0000 L CNN
+F 2 "TO_SOT_Packages_SMD:SOT-23_Handsoldering" V 5350 3550 50  0001 C CNN
 F 3 "" V 5350 3550 50  0000 C CNN
 	1    5350 3550
@@
 F 0 "C307" H 4960 4070 50  0000 L CNN
 F 1 "1nF" H 4960 3920 50  0000 L CNN
-F 2 "" H 4950 4000 50  0000 C CNN
+F 2 "Capacitors_SMD:C_0805" H 4950 4000 50  0001 C CNN
 F 3 "" H 4950 4000 50  0000 C CNN
 	1    4950 4000
@@
 F 0 "C308" H 5360 4070 50  0000 L CNN
 F 1 "1nF" H 5360 3920 50  0000 L CNN
-F 2 "" H 5350 4000 50  0000 C CNN
+F 2 "Capacitors_SMD:C_0805" H 5350 4000 50  0001 C CNN
 F 3 "" H 5350 4000 50  0000 C CNN
 	1    5350 4000
@@
 F 0 "C309" H 5660 4070 50  0000 L CNN
 F 1 "100nF" H 5660 3920 50  0000 L CNN
-F 2 "" H 5650 4000 50  0000 C CNN
+F 2 "Capacitors_SMD:C_0805" H 5650 4000 50  0001 C CNN
 F 3 "" H 5650 4000 50  0000 C CNN
 	1    5650 4000
@@
 F 0 "C306" H 4660 4070 50  0000 L CNN
 F 1 "100nF" H 4660 3920 50  0000 L CNN
-F 2 "" H 4650 4000 50  0000 C CNN
+F 2 "Capacitors_SMD:C_0805" H 4650 4000 50  0001 C CNN
 F 3 "" H 4650 4000 50  0000 C CNN
 	1    4650 4000
@@
 $EndComp
 $Comp
-L +Vlogic #PWR302
+L +Vlogic #PWR014
 U 1 1 57E32A6B
 P 4100 3900
-F 0 "#PWR302" H 4100 3700 50  0001 C CNN
+F 0 "#PWR014" H 4100 3700 50  0001 C CNN
 F 1 "+Vlogic" H 4100 4100 50  0000 C CNN
 F 2 "" H 4100 3900 50  0000 C CNN
@@
 $EndComp
 $Comp
-L GND #PWR304
+L GND #PWR015
 U 1 1 57E32A71
 P 5150 4300
-F 0 "#PWR304" H 5150 4050 50  0001 C CNN
+F 0 "#PWR015" H 5150 4050 50  0001 C CNN
 F 1 "GND" H 5150 4150 50  0000 C CNN
 F 2 "" H 5150 4300 50  0000 C CNN
@@
 Connection ~ 5350 3800
 $Comp
-L GND #PWR303
+L GND #PWR016
 U 1 1 57E32AAA
 P 4400 4400
-F 0 "#PWR303" H 4400 4150 50  0001 C CNN
+F 0 "#PWR016" H 4400 4150 50  0001 C CNN
 F 1 "GND" H 4400 4250 50  0000 C CNN
 F 2 "" H 4400 4400 50  0000 C CNN
@@
 F 0 "L303" H 7230 3240 50  0000 L CNN
 F 1 "1µ6" H 7230 3160 50  0000 L CNN
-F 2 "" H 7200 3200 50  0000 C CNN
+F 2 "" H 7200 3200 50  0001 C CNN
 F 3 "" H 7200 3200 50  0000 C CNN
 	1    7200 3200
@@
 F 0 "D304" H 7150 3630 50  0000 L CNN
 F 1 "1N4007" H 7050 3470 50  0000 L CNN
-F 2 "" V 7200 3550 50  0000 C CNN
+F 2 "" V 7200 3550 50  0001 C CNN
 F 3 "" V 7200 3550 50  0000 C CNN
 	1    7200 3550
@@
 F 0 "R304" H 6930 3570 50  0000 L CNN
 F 1 "100k" H 6930 3510 50  0000 L CNN
-F 2 "" H 6900 3550 50  0000 C CNN
+F 2 "Resistors_SMD:R_0805_HandSoldering" H 6900 3550 50  0001 C CNN
 F 3 "" H 6900 3550 50  0000 C CNN
 	1    6900 3550
@@
 F 0 "C311" H 7860 3520 50  0000 L CNN
 F 1 "330pF" H 7860 3370 50  0000 L CNN
-F 2 "" H 7850 3450 50  0000 C CNN
+F 2 "Capacitors_SMD:C_0805" H 7850 3450 50  0001 C CNN
 F 3 "" H 7850 3450 50  0000 C CNN
 	1    7850 3450
@@
 F 0 "D305" H 7400 3180 50  0000 L CNN
 F 1 "1N4007" H 7300 3020 50  0000 L CNN
-F 2 "" V 7450 3100 50  0000 C CNN
+F 2 "" V 7450 3100 50  0001 C CNN
 F 3 "" V 7450 3100 50  0000 C CNN
 	1    7450 3100
@@
 F 0 "R305" H 7680 2970 50  0000 L CNN
 F 1 "100R" H 7680 2910 50  0000 L CNN
-F 2 "" H 7650 2950 50  0000 C CNN
+F 2 "Resistors_SMD:R_0805_HandSoldering" H 7650 2950 50  0001 C CNN
 F 3 "" H 7650 2950 50  0000 C CNN
 	1    7650 2950
@@
 F 0 "C310" H 7860 3170 50  0000 L CNN
 F 1 "10nF" H 7860 3020 50  0000 L CNN
-F 2 "" H 7850 3100 50  0000 C CNN
+F 2 "Capacitors_SMD:C_0805" H 7850 3100 50  0001 C CNN
 F 3 "" H 7850 3100 50  0000 C CNN
 	1    7850 3100
@@
 Connection ~ 6900 3450
 $Comp
-L GND #PWR305
+L GND #PWR017
 U 1 1 57E32AFA
 P 7400 3750
-F 0 "#PWR305" H 7400 3500 50  0001 C CNN
+F 0 "#PWR017" H 7400 3500 50  0001 C CNN
 F 1 "GND" H 7400 3600 50  0000 C CNN
 F 2 "" H 7400 3750 50  0000 C CNN
@@
 F 0 "L304" V 8000 2850 50  0000 C CNN
 F 1 "10µH" V 8150 2850 50  0000 C CNN
-F 2 "" H 8050 2850 50  0000 C CNN
+F 2 "" H 8050 2850 50  0001 C CNN
 F 3 "" H 8050 2850 50  0000 C CNN
 	1    8050 2850

Commit message: Changed SWR microstrip for two transformers and gave missing values for components
Parts:
- removed LINE301: microstrip, symbol microstrip
- added D306: BAP65-02, symbol D_Small
- added R? (x4): 1k, symbol R
- added T? (x2): TRANSFO, symbol TRANSFO
- D304, D305: value 1N4007 -> BAP65-02
Connections:
- wire segments 51 -> 65
Other:
- moved on the sheet: C306, C307, C308, C309, D301, D302, D303, D304, R301, R302, R303
