File: hardware/tx_chain.sch (KiCad schematic (older format))
At the start: 34 parts, among them Q501 BCP56, Q502 IRL510, T501 TRANSFO2, U501 74LVC1G3157, U502 74LVC1G3157

Commit message: Fixed some bugs and annotated rest of the footprints
Parts:
- C501: footprint Capacitors_SMD:C_0805 -> dodekaedri:CAP_6.3x5.8mm
- C502, C503, C504, C505, C506, C507, C508, C509, C510, C511, C512, C513: footprint Capacitors_SMD:C_0805 -> Capacitors_SMD:C_0805_HandSoldering
- D501: footprint (none) -> LEDs:LED_0805
- FB501: footprint (none) -> Resistors_SMD:R_0805_HandSoldering
- L501, L502, L503: footprint (none) -> Air_Coils_SML_NEOSID:Neosid_Air-Coil_SML_5turn_HDM0531A
- Q501: footprint (none) -> TO_SOT_Packages_SMD:SOT-223
- Q502: footprint (none) -> TO_SOT_Packages_THT:TO-220_Neutral123_Vertical
- T501: footprint (none) -> dodekaedri:transf_5_pin
- U501, U502: footprint (none) -> TO_SOT_Packages_SMD:SOT-23-6_Handsoldering
Changed lines of the file:
@@
 F 0 "U501" H 2650 3600 60  0000 C CNN
 F 1 "74LVC1G3157" H 2650 4100 60  0000 C CNN
-F 2 "" H 2650 3750 60  0001 C CNN
+F 2 "TO_SOT_Packages_SMD:SOT-23-6_Handsoldering" H 2650 3750 60  0001 C CNN
 F 3 "" H 2650 3750 60  0001 C CNN
 	1    2650 3850
@@
 F 0 "U502" H 2650 4300 60  0000 C CNN
 F 1 "74LVC1G3157" H 2650 4800 60  0000 C CNN
-F 2 "" H 2650 4450 60  0001 C CNN
+F 2 "TO_SOT_Packages_SMD:SOT-23-6_Handsoldering" H 2650 4450 60  0001 C CNN
 F 3 "" H 2650 4450 60  0001 C CNN
 	1    2650 4550
@@
 $EndComp
 $Comp
-L GND #PWR503
+L GND #PWR021
 U 1 1 57E4343C
 P 3100 4100
-F 0 "#PWR503" H 3100 3850 50  0001 C CNN
+F 0 "#PWR021" H 3100 3850 50  0001 C CNN
 F 1 "GND" H 3100 3950 50  0000 C CNN
 F 2 "" H 3100 4100 50  0000 C CNN
@@
 $EndComp
 $Comp
-L GND #PWR504
+L GND #PWR022
 U 1 1 57E4345E
 P 3100 4800
-F 0 "#PWR504" H 3100 4550 50  0001 C CNN
+F 0 "#PWR022" H 3100 4550 50  0001 C CNN
 F 1 "GND" H 3100 4650 50  0000 C CNN
 F 2 "" H 3100 4800 50  0000 C CNN
@@
 $EndComp
 $Comp
-L +Vlogic #PWR501
+L +Vlogic #PWR023
 U 1 1 57E434AC
 P 2150 3550
-F 0 "#PWR501" H 2150 3350 50  0001 C CNN
+F 0 "#PWR023" H 2150 3350 50  0001 C CNN
 F 1 "+Vlogic" H 2150 3750 50  0000 C CNN
 F 2 "" H 2150 3550 50  0000 C CNN
@@
 $EndComp
 $Comp
-L +Vlogic #PWR502
+L +Vlogic #PWR024
 U 1 1 57E434C4
 P 2150 4250
-F 0 "#PWR502" H 2150 4050 50  0001 C CNN
+F 0 "#PWR024" H 2150 4050 50  0001 C CNN
 F 1 "+Vlogic" H 2150 4450 50  0000 C CNN
 F 2 "" H 2150 4250 50  0000 C CNN
@@
 F 0 "T501" H 4350 4750 50  0000 C CNN
 F 1 "TRANSFO2" H 4350 3750 50  0000 C CNN
-F 2 "" H 4350 4250 50  0001 C CNN
+F 2 "dodekaedri:transf_5_pin" H 4350 4250 50  0001 C CNN
 F 3 "" H 4350 4250 50  0000 C CNN
 	1    4350 4250
@@
 F 0 "C501" H 3450 4450 50  0000 L CNN
 F 1 "220µF" V 3500 3950 50  0000 L CNN
-F 2 "Capacitors_SMD:C_0805" H 3588 4100 50  0001 C CNN
+F 2 "dodekaedri:CAP_6.3x5.8mm" H 3588 4100 50  0001 C CNN
 F 3 "" H 3550 4250 50  0000 C CNN
 	1    3550 4250
@@
 F 0 "C502" H 3700 4450 50  0000 L CNN
 F 1 "100nF" H 3775 4150 50  0000 L CNN
-F 2 "Capacitors_SMD:C_0805" H 3788 4100 50  0001 C CNN
+F 2 "Capacitors_SMD:C_0805_HandSoldering" H 3788 4100 50  0001 C CNN
 F 3 "" H 3750 4250 50  0000 C CNN
 	1    3750 4250
@@
 $EndComp
 $Comp
-L GND #PWR505
+L GND #PWR025
 U 1 1 57E43B57
 P 3650 4450
-F 0 "#PWR505" H 3650 4200 50  0001 C CNN
+F 0 "#PWR025" H 3650 4200 50  0001 C CNN
 F 1 "GND" H 3650 4300 50  0000 C CNN
 F 2 "" H 3650 4450 50  0000 C CNN
@@
 $EndComp
 $Comp
-L GND #PWR506
+L GND #PWR026
 U 1 1 57E43B98
 P 5100 4800
-F 0 "#PWR506" H 5100 4550 50  0001 C CNN
+F 0 "#PWR026" H 5100 4550 50  0001 C CNN
 F 1 "GND" H 5100 4650 50  0000 C CNN
 F 2 "" H 5100 4800 50  0000 C CNN
@@
 F 0 "L501" V 5250 4050 50  0000 C CNN
 F 1 "1µH" V 5400 4050 50  0000 C CNN
-F 2 "" H 5300 4050 50  0001 C CNN
+F 2 "Air_Coils_SML_NEOSID:Neosid_Air-Coil_SML_5turn_HDM0531A" H 5300 4050 50  0001 C CNN
 F 3 "" H 5300 4050 50  0000 C CNN
 	1    5300 4050
@@
 F 0 "C503" H 5725 4400 50  0000 L CNN
 F 1 "330pF" H 5725 4200 50  0000 L CNN
-F 2 "Capacitors_SMD:C_0805" H 5738 4150 50  0001 C CNN
+F 2 "Capacitors_SMD:C_0805_HandSoldering" H 5738 4150 50  0001 C CNN
 F 3 "" H 5700 4300 50  0000 C CNN
 	1    5700 4300
@@
 F 0 "C504" H 5975 4150 50  0000 L CNN
 F 1 "10nF" H 5975 3950 50  0000 L CNN
-F 2 "Capacitors_SMD:C_0805" H 5988 3900 50  0001 C CNN
+F 2 "Capacitors_SMD:C_0805_HandSoldering" H 5988 3900 50  0001 C CNN
 F 3 "" H 5950 4050 50  0000 C CNN
 	1    5950 4050
@@
 F 0 "Q501" H 6850 4100 50  0000 R CNN
 F 1 "BCP56" H 6900 4000 50  0000 R CNN
-F 2 "" H 6700 4150 50  0001 C CNN
+F 2 "TO_SOT_Packages_SMD:SOT-223" H 6700 4150 50  0001 C CNN
 F 3 "" H 6500 4050 50  0000 C CNN
 	1    6500 4050
@@
 $EndComp
 $Comp
-L GND #PWR508
+L GND #PWR027
 U 1 1 57E44284
 P 6600 4800
-F 0 "#PWR508" H 6600 4550 50  0001 C CNN
+F 0 "#PWR027" H 6600 4550 50  0001 C CNN
 F 1 "GND" H 6600 4650 50  0000 C CNN
 F 2 "" H 6600 4800 50  0000 C CNN
@@
 F 0 "C505" H 6875 3450 50  0000 L CNN
 F 1 "100nF" H 6875 3250 50  0000 L CNN
-F 2 "Capacitors_SMD:C_0805" H 6888 3200 50  0001 C CNN
+F 2 "Capacitors_SMD:C_0805_HandSoldering" H 6888 3200 50  0001 C CNN
 F 3 "" H 6850 3350 50  0000 C CNN
 	1    6850 3350
@@
 $EndComp
 $Comp
-L GND #PWR509
+L GND #PWR028
 U 1 1 57E451F7
 P 6850 3550
-F 0 "#PWR509" H 6850 3300 50  0001 C CNN
+F 0 "#PWR028" H 6850 3300 50  0001 C CNN
 F 1 "GND" H 6850 3400 50  0000 C CNN
 F 2 "" H 6850 3550 50  0000 C CNN
@@
 F 0 "C506" H 7225 3900 50  0000 L CNN
 F 1 "10nF" H 7225 3700 50  0000 L CNN
-F 2 "Capacitors_SMD:C_0805" H 7238 3650 50  0001 C CNN
+F 2 "Capacitors_SMD:C_0805_HandSoldering" H 7238 3650 50  0001 C CNN
 F 3 "" H 7200 3800 50  0000 C CNN
 	1    7200 3800
@@
 F 0 "C507" H 7725 3900 50  0000 L CNN
 F 1 "10nF" H 7725 3700 50  0000 L CNN
-F 2 "Capacitors_SMD:C_0805" H 7738 3650 50  0001 C CNN
+F 2 "Capacitors_SMD:C_0805_HandSoldering" H 7738 3650 50  0001 C CNN
 F 3 "" H 7700 3800 50  0000 C CNN
 	1    7700 3800
@@
 F 0 "Q502" H 8650 3850 50  0000 R CNN
 F 1 "IRL510" H 8700 3750 50  0000 R CNN
-F 2 "" H 8450 3900 50  0001 C CNN
+F 2 "TO_SOT_Packages_THT:TO-220_Neutral123_Vertical" H 8450 3900 50  0001 C CNN
 F 3 "" H 8250 3800 50  0000 C CNN
 	1    8250 3800
@@
 F 0 "L502" V 8300 3100 50  0000 C CNN
 F 1 "1µH" V 8450 3100 50  0000 C CNN
-F 2 "" H 8350 3100 50  0001 C CNN
+F 2 "Air_Coils_SML_NEOSID:Neosid_Air-Coil_SML_5turn_HDM0531A" H 8350 3100 50  0001 C CNN
 F 3 "" H 8350 3100 50  0000 C CNN
 	1    8350 3100
@@
 F 0 "C509" H 8025 3050 50  0000 L CNN
 F 1 "100nF" H 8025 2850 50  0000 L CNN
-F 2 "Capacitors_SMD:C_0805" H 8038 2800 50  0001 C CNN
+F 2 "Capacitors_SMD:C_0805_HandSoldering" H 8038 2800 50  0001 C CNN
 F 3 "" H 8000 2950 50  0000 C CNN
 	1    8000 2950
@@
 $EndComp
 $Comp
-L GND #PWR511
+L GND #PWR029
 U 1 1 57E458EE
 P 8000 3150
-F 0 "#PWR511" H 8000 2900 50  0001 C CNN
+F 0 "#PWR029" H 8000 2900 50  0001 C CNN
 F 1 "GND" H 8000 3000 50  0000 C CNN
 F 2 "" H 8000 3150 50  0000 C CNN
@@
 $EndComp
 $Comp
-L Vin #Vin501
+L Vin #Vin030
 U 1 1 57E45ADD
 P 8350 2100
-F 0 "#Vin501" H 8500 2150 60  0001 C CNN
+F 0 "#Vin030" H 8500 2150 60  0001 C CNN
 F 1 "Vin" H 8200 2150 60  0000 C CNN
 F 2 "" H 8350 2100 60  0001 C CNN
@@
 $EndComp
 $Comp
-L GND #PWR512
+L GND #PWR031
 U 1 1 57E45E2D
 P 8350 4900
-F 0 "#PWR512" H 8350 4650 50  0001 C CNN
+F 0 "#PWR031" H 8350 4650 50  0001 C CNN
 F 1 "GND" H 8350 4750 50  0000 C CNN
 F 2 "" H 8350 4900 50  0000 C CNN
@@
 F 0 "L503" V 9450 3500 50  0000 C CNN
 F 1 "800nH" V 9600 3500 50  0000 C CNN
-F 2 "" H 9500 3500 50  0001 C CNN
+F 2 "Air_Coils_SML_NEOSID:Neosid_Air-Coil_SML_5turn_HDM0531A" H 9500 3500 50  0001 C CNN
 F 3 "" H 9500 3500 50  0000 C CNN
 	1    9500 3500
@@
 F 0 "C512" H 9125 3850 50  0000 L CNN
 F 1 "330pF" H 9125 3650 50  0000 L CNN
-F 2 "Capacitors_SMD:C_0805" H 9138 3600 50  0001 C CNN
+F 2 "Capacitors_SMD:C_0805_HandSoldering" H 9138 3600 50  0001 C CNN
 F 3 "" H 9100 3750 50  0000 C CNN
 	1    9100 3750
@@
 F 0 "C513" H 9925 3850 50  0000 L CNN
 F 1 "1nF" H 9925 3650 50  0000 L CNN
-F 2 "Capacitors_SMD:C_0805" H 9938 3600 50  0001 C CNN
+F 2 "Capacitors_SMD:C_0805_HandSoldering" H 9938 3600 50  0001 C CNN
 F 3 "" H 9900 3750 50  0000 C CNN
 	1    9900 3750
@@
 $EndComp
 $Comp
-L GND #PWR515
+L GND #PWR032
 U 1 1 57E465CB
 P 9500 4100
-F 0 "#PWR515" H 9500 3850 50  0001 C CNN
+F 0 "#PWR032" H 9500 3850 50  0001 C CNN
 F 1 "GND" H 9500 3950 50  0000 C CNN
 F 2 "" H 9500 4100 50  0000 C CNN
@@
 $EndComp
 $Comp
-L GND #PWR507
+L GND #PWR033
 U 1 1 57E471D5
 P 5700 3800
-F 0 "#PWR507" H 5700 3550 50  0001 C CNN
+F 0 "#PWR033" H 5700 3550 50  0001 C CNN
 F 1 "GND" H 5700 3650 50  0000 C CNN
 F 2 "" H 5700 3800 50  0000 C CNN
@@
 F 0 "C511" H 8875 4850 50  0000 L CNN
 F 1 "10nF" H 8875 4650 50  0000 L CNN
-F 2 "Capacitors_SMD:C_0805" H 8888 4600 50  0001 C CNN
+F 2 "Capacitors_SMD:C_0805_HandSoldering" H 8888 4600 50  0001 C CNN
 F 3 "" H 8850 4750 50  0000 C CNN
 	1    8850 4750
@@
 F 0 "C508" H 7750 5500 50  0000 L CNN
 F 1 "10nF" H 7975 5300 50  0000 L CNN
-F 2 "Capacitors_SMD:C_0805" H 7988 5250 50  0001 C CNN
+F 2 "Capacitors_SMD:C_0805_HandSoldering" H 7988 5250 50  0001 C CNN
 F 3 "" H 7950 5400 50  0000 C CNN
 	1    7950 5400
@@
 $EndComp
 $Comp
-L GND #PWR510
+L GND #PWR034
 U 1 1 57EBA5D8
 P 7950 5550
-F 0 "#PWR510" H 7950 5300 50  0001 C CNN
+F 0 "#PWR034" H 7950 5300 50  0001 C CNN
 F 1 "GND" H 7950 5400 50  0000 C CNN
 F 2 "" H 7950 5550 50  0000 C CNN
@@
 F 0 "C510" H 8575 5500 50  0000 L CNN
 F 1 "10nF" H 8575 5300 50  0000 L CNN
-F 2 "Capacitors_SMD:C_0805" H 8588 5250 50  0001 C CNN
+F 2 "Capacitors_SMD:C_0805_HandSoldering" H 8588 5250 50  0001 C CNN
 F 3 "" H 8550 5400 50  0000 C CNN
 	1    8550 5400
@@
 $EndComp
 $Comp
-L GND #PWR513
+L GND #PWR035
 U 1 1 57EBA6B5
 P 8550 5600
-F 0 "#PWR513" H 8550 5350 50  0001 C CNN
+F 0 "#PWR035" H 8550 5350 50  0001 C CNN
 F 1 "GND" H 8550 5450 50  0000 C CNN
 F 2 "" H 8550 5600 50  0000 C CNN
@@
 F 0 "FB501" H 8350 2600 50  0000 C CNN
 F 1 "FILTER" H 8350 2350 50  0000 C CNN
-F 2 "" H 8350 2450 50  0001 C CNN
+F 2 "Resistors_SMD:R_0805_HandSoldering" H 8350 2450 50  0001 C CNN
 F 3 "" H 8350 2450 50  0000 C CNN
 	1    8350 2450
@@
 $EndComp
 $Comp
-L GND #PWR514
+L GND #PWR036
 U 1 1 57EAC40D
 P 9100 5600
-F 0 "#PWR514" H 9100 5350 50  0001 C CNN
+F 0 "#PWR036" H 9100 5350 50  0001 C CNN
 F 1 "GND" H 9100 5450 50  0000 C CNN
 F 2 "" H 9100 5600 50  0000 C CNN
@@
 	9100 5600 9100 5550
 $Comp
-L PWR_FLAG #FLG501
+L PWR_FLAG #FLG037
 U 1 1 57EE999B
 P 8750 2100
-F 0 "#FLG501" H 8750 2195 50  0001 C CNN
+F 0 "#FLG037" H 8750 2195 50  0001 C CNN
 F 1 "PWR_FLAG" H 8750 2280 50  0000 C CNN
 F 2 "" H 8750 2100 50  0000 C CNN
@@
 F 0 "D501" H 5700 3700 50  0000 C CNN
 F 1 "RED" H 5700 3450 50  0000 C CNN
-F 2 "" H 5700 3600 50  0000 C CNN
+F 2 "LEDs:LED_0805" H 5700 3600 50  0001 C CNN
 F 3 "" H 5700 3600 50  0000 C CNN
 	1    5700 3600
