File: hardware/psu.sch (KiCad schematic (older format))
At the start: 17 parts, among them CON401 BARREL_JACK, U401 NCP3170-D

Commit message: halfway through layout
Connections:
- net Vin_connector renamed Vin_net
Changed lines of the file:
@@
 Connection ~ 3700 4200
 Connection ~ 3100 2950
+$Comp
+L Vin #Vin021
+U 1 1 57F50F83
+P 3350 2600
+F 0 "#Vin021" H 3500 2650 60  0001 C CNN
+F 1 "Vin" H 3200 2650 60  0000 C CNN
+F 2 "" H 3350 2600 60  0001 C CNN
+F 3 "" H 3350 2600 60  0001 C CNN
+	1    3350 2600
+	1    0    0    -1
+$EndComp
 $EndSCHEMATC
