File: hardware/dodekaedri.kicad_pcb (KiCad board)
At the start: 4 copper layers, 76.2 x 76.2 mm, 237 parts, among them CON401 BARREL_JACK, J801 HANDSFREE, J802 microphone, J803 HEADPHONES, P301 BNC, P801 TX_SW_WIRE, P802 USB_OTG, P803 UART, P804 PROG, P805 RNG_PINS, P806 CONN_01X08, P807 CONN_01X04, P808 CONN_02X04, P809 BOOT0JMPR, Q501 BCP56, Q502 IRL510, Q801 BSS84, SW801 SW_PUSH, SW802 SW, SW803 SW, SW804 SW, SW805 SW, SW806 encoder, SW807 RESET, SW808 SW, SW809 encoder, SW810 SW, T301 TRANSFO, T302 TRANSFO, T501 TRANSFO2, T601 TRANSFO2, U201 MIC5365, U202 SI5351A, U401 NCP3170-D, U501 74LVC1G3157, U502 74LVC1G3157, U601 74LVC1G3157, U602 74LVC1G3157, U603 TL972IDR, U701 WM8731, U702 MCP6L02, U801 STM32F401, U802 WM8731

Commit message: save layout _before_ doing drastinc netlist changes
Parts:
- removed J802: microphone, dodekaedri:TRS_jack
- removed J803: HEADPHONES, dodekaedri:TRS_jack
- removed SW805, SW808, SW810: SW, Buttons_Switches_SMD:SW_SPST_B3SL-1002P
- removed SW809: encoder, dodekaedri:encoder
- D802: footprint Diodes_SMD:SOD-523 -> Diodes_SMD:D_0805
- P802: moved to B.Cu
- moved P804 142.7 mm to (109.2, 94.0), turned to 90 degrees
- moved P802 129.9 mm to (188.7, 93.0), turned to 270 degrees
- moved P803 128.5 mm to (111.8, 99.1), turned to 90 degrees
- moved J801 88.3 mm to (174.0, 100.3), turned to 135 degrees
- moved P801 58.9 mm to (123.2, 109.2), turned to 135 degrees
- moved P805 46.7 mm to (109.2, 71.1), turned to 0 degrees
- moved Q502 42.4 mm to (146.1, 50.2), turned to 0 degrees
- moved P301 34.5 mm to (133.3, 54.6), turned to 0 degrees
- moved SW803 26.0 mm to (133.6, 101.6)
- moved SW807 24.1 mm to (119.4, 64.8)
- moved P806 17.0 mm to (116.8, 71.1)
- moved R309 16.9 mm to (256.5, 134.6)
- moved SW801 15.3 mm to (128.3, 116.8), turned to 135 degrees
- moved SW806 13.9 mm to (156.8, 109.2)
- moved SW804 12.2 mm to (143.3, 101.6)
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Routing:
- net GND: track 41.2 -> 59.0 mm, vias 0 -> 1
Other:
- board size 76.2 x 76.2 mm -> 336.6 x 85.1 mm
- net class Default: via_dia 0.7 -> 0.8; via_drill 0.6 -> 0.5
- net class thicker_track removed
- rule via_min_drill: 0.6 -> 0.5
- rule via_min_size: 0.7 -> 0.8
- board text added: "PROG"
- board text added: "RX SWITCH"
- board text added: "UART"

Commit message: 15% of layout done.. hopefully
Parts:
- added C514: 1nF, Capacitors_SMD:C_0805_HandSoldering, F.Cu at (25.9, 142.7)
- added C515: 1nF, Capacitors_SMD:C_0805_HandSoldering, F.Cu at (25.7, 136.7)
- added R512: 100R, Resistors_SMD:R_0805_HandSoldering, F.Cu at (33.8, 133.6)
- added R513: 100R, Resistors_SMD:R_0805_HandSoldering, F.Cu at (35.3, 138.7)
- C601, C602, C603, C604, C605, C606, C607, L601, L602, L603, L604, R601, R602, R603, R604, R605, R606, T601, U601, U602: moved to B.Cu
- U701, U802: moved to F.Cu
- moved C702 255.0 mm to (154.7, 74.9)
- moved C701 250.5 mm to (153.0, 80.1), turned to 90 degrees
- moved C602 192.1 mm to (152.1, 66.3), turned to 180 degrees
- moved C604 191.5 mm to (152.3, 63.9)
- moved R603 189.6 mm to (152.3, 61.6)
- moved C606 187.6 mm to (161.7, 63.2)
- moved C603 184.6 mm to (157.1, 81.2), turned to 270 degrees
- moved R605 183.9 mm to (157.9, 67.4), turned to 90 degrees
- moved L601 183.7 mm to (146.9, 68.7), turned to 180 degrees
- moved C605 182.8 mm to (161.0, 81.2), turned to 270 degrees
- moved C601 182.8 mm to (156.1, 71.6), turned to 180 degrees
- moved L603 182.1 mm to (146.9, 65.7)
- moved R601 181.6 mm to (152.3, 68.7)
- moved L604 180.8 mm to (149.6, 84.3)
- moved C607 178.2 mm to (168.8, 67.8), turned to 90 degrees
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Connections:
- R825 pad 2: /CPU/PC13 -> /CPU/PC14
- R826 pad 2: /CPU/PC15 -> /CPU/PC13
- R827 pad 2: /CPU/PH0 -> /CPU/PC15
- U501 pad 4: /TX_chain/TX_I -> Net-(R512-Pad1)
- U502 pad 4: /TX_chain/TX_Q -> Net-(R513-Pad1)
- U801 pad 3: /CPU/CLK_CPU -> /CPU/PC14
- U801 pad 5: /CPU/PH0 -> /CPU/CLK_CPU
Routing:
- net /RX_chain/RX_BIAS: track 0.00 -> 49.4 mm
- net /RX_chain/RX_Q: track 0.00 -> 25.1 mm, vias 0 -> 1
- net Net-(C607-Pad2): track 0.00 -> 21.9 mm
- net Net-(C606-Pad1): track 0.00 -> 19.0 mm
- net /CPU/RFLRC: track 0.00 -> 18.2 mm
- net /CPU/RFADCDAT: track 0.00 -> 14.1 mm
- net Net-(C605-Pad2): track 0.00 -> 13.8 mm
- net /CPU/RFDACDAT: track 0.00 -> 12.8 mm
- net /RX_chain/RX_I: track 0.00 -> 11.9 mm
- net Net-(T601-Pad3): track 0.00 -> 11.4 mm
- net Net-(T601-Pad6): track 0.00 -> 11.0 mm
- net /CPU/RFBCLK: track 0.00 -> 10.9 mm, vias 0 -> 2
- net +Vlogic: track 24.0 -> 34.5 mm, vias 0 -> 5
- net /RX_chain/LO_I: track 0.00 -> 10.0 mm
- net Net-(L601-Pad1): track 0.00 -> 8.78 mm
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
Commit message: halfway through layout
Parts:
- removed C303: 3nF, Capacitors_SMD:C_0805_HandSoldering
- removed D601, D602: BAP65-02, Diodes_SMD:SOD-523
- removed D808, D811, D813, D815, D816, D817: 1N914, TO_SOT_Packages_SMD:SOT-23_Handsoldering
- removed L302: 660nH, Air_Coils_SML_NEOSID:Neosid_Air-Coil_SML_5turn_HDM0531A
- removed R817, R829: 50R, Resistors_SMD:R_0805_HandSoldering
- added C608: 100nF, Capacitors_SMD:C_0805_HandSoldering, F.Cu at (14.3, 127.9)
- added R704: 0R, Resistors_SMD:R_0805_HandSoldering, F.Cu at (158.8, 69.3)
- added R705: 0R, Resistors_SMD:R_0805_HandSoldering, F.Cu at (160.9, 62.5)
- added R822: 10k, Resistors_SMD:R_0805_HandSoldering, F.Cu at (14.4, 138.7)
- C301, C302, C304, C305, C403, C508, C510, C511, C512, D401, FB401, L301, R401, R506, R507, R509, R510, R511, R703: moved to B.Cu
- C606, C607: value 100pF -> 1nF
- D301, D302, D303, D805, D806, D807, D809, D810, D812: footprint TO_SOT_Packages_SMD:SOT-23_Handsoldering -> dodekaedri:SOT-23_HS_2-1-3
- L304: value 10µH -> 470µH; footprint Resistors_SMD:R_0805_HandSoldering -> dodekaedri:SMT_1007
- R605, R606: value 33k -> 1k
- R808: value 47k -> 100k
- R813: value 1k -> 100k
- R815: value 680R -> 1k
- U702: moved to F.Cu
- moved D812 321.6 mm to (8.13, 130.2)
- moved D807 304.4 mm to (14.5, 117.3)
- moved D809 300.3 mm to (33.6, 121.8)
- moved R511 278.9 mm to (119.6, 59.1), turned to 45 degrees
- moved R507 278.8 mm to (118.9, 64.0), turned to 135 degrees
- moved R510 276.8 mm to (116.0, 64.8), turned to 315 degrees
- moved D806 271.6 mm to (28.1, 118.9)
- moved R509 267.2 mm to (136.8, 50.7), turned to 180 degrees
- moved C510 260.5 mm to (121.9, 61.6), turned to 45 degrees
- moved D805 257.2 mm to (21.2, 120.3)
- moved C513 256.7 mm to (136.1, 62.5), turned to 180 degrees
- moved D810 255.8 mm to (33.6, 113.3)
- moved C511 255.7 mm to (132.6, 52.1), turned to 270 degrees
- moved U501 252.6 mm to (133.0, 86.4)
- moved C508 252.2 mm to (136.9, 57.8), turned to 180 degrees
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Connections:
- C401 pad 1: /PSU/Vin_connector -> Vin_net
- CON401 pad 1: /PSU/Vin_connector -> Vin_net
- D401 pad 1: /PSU/Vin_connector -> Vin_net
- D802 pad 1: Net-(D802-Pad1) -> Vin_net
- D823 pad 3: /CPU/PC3 -> /CPU/VIN_ADC
- FB401 pad 1: /PSU/Vin_connector -> Vin_net
- FB501 pad 1: Net-(FB501-Pad1) -> Vin_net
- L301 pad 2: Net-(C303-Pad1) -> Net-(C304-Pad1)
- P805 pad 3: Net-(P805-Pad3) -> GND
- R813 pad 1: Net-(P808-Pad6) -> Vin_net
- R813 pad 2: Net-(R813-Pad2) -> /CPU/VIN_ADC
- U702 pad 1: /TX_chain/TX_BIAS -> Net-(R704-Pad2)
- U702 pad 2: /TX_chain/TX_BIAS -> Net-(R704-Pad2)
- U702 pad 6: /RX_chain/RX_BIAS -> Net-(R705-Pad2)
- U702 pad 7: /RX_chain/RX_BIAS -> Net-(R705-Pad2)
- U801 pad 11: /CPU/PC3 -> /CPU/VIN_ADC
Routing:
- net GND: track 63.1 -> 140.9 mm, vias 10 -> 16
- net /CPU/PA_BIAS: track 0.00 -> 53.4 mm, vias 0 -> 2
- net Net-(R818-Pad1): track 0.00 -> 33.3 mm, vias 0 -> 2
- net Net-(C402-Pad2): track 0.00 -> 32.5 mm, vias 0 -> 1
- net +Vlogic: track 34.5 -> 62.8 mm, vias 5 -> 11
- net Net-(C508-Pad1): track 0.00 -> 27.5 mm, vias 0 -> 2
- net Net-(Q502-Pad3): track 0.00 -> 16.8 mm
- net /TX_chain/TX_Q: track 0.00 -> 15.0 mm, vias 0 -> 2
- net /RX_chain/RX_I: track 11.9 -> 24.5 mm, vias 0 -> 1
- net /CPU/I2S_MCLK: track 0.00 -> 12.3 mm
- net Net-(C404-Pad1): track 0.00 -> 12.0 mm
- net Net-(C301-Pad1): track 0.00 -> 11.5 mm
- net Net-(C605-Pad2): track 13.8 -> 2.78 mm
- net /TX_chain/TX_I: track 0.00 -> 10.9 mm, vias 0 -> 2
- net Net-(C512-Pad1): track 0.00 -> 8.90 mm, vias 0 -> 1
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
Commit message: one fourth to go... area-wise :D
Parts:
- C311, C506, C812, C813, C814, C815, C816, C817, C818, C819, D301, D302, D303, D304, D305, D306, FB801, FB803, L303, R304, R305, R810, R811, R812, R816, R820, R821, T301, T302, U802: moved to B.Cu
- moved C502 270.5 mm to (132.6, 68.1), turned to 90 degrees
- moved C703 241.7 mm to (166.8, 89.3), turned to 135 degrees
- moved C704 231.3 mm to (164.5, 90.0), turned to 135 degrees
- moved C501 230.5 mm to (128.3, 64.8), turned to 180 degrees
- moved R307 222.2 mm to (81.3, 67.8)
- moved R306 216.7 mm to (79.2, 64.5)
- moved C308 215.7 mm to (72.9, 59.2)
- moved R301 213.8 mm to (72.6, 66.0)
- moved R304 212.7 mm to (91.2, 51.3), turned to 180 degrees
- moved T501 212.7 mm to (137.0, 68.1), turned to 90 degrees
- moved C809 209.1 mm to (150.5, 93.6), turned to 270 degrees
- moved C805 207.1 mm to (136.4, 78.1), turned to 45 degrees
- moved C807 206.4 mm to (136.8, 75.1), turned to 45 degrees
- moved C306 205.1 mm to (79.8, 58.7)
- moved R309 202.3 mm to (67.8, 61.7)
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Routing:
- net GND: track 140.9 -> 258.1 mm, vias 16 -> 22
- net /CPU/I2C1_SDA: track 4.62 -> 97.4 mm, vias 0 -> 4
- net /CPU/I2C1_CLK: track 7.06 -> 89.1 mm, vias 0 -> 4
- net +Vlogic: track 62.8 -> 116.1 mm
- net Net-(C819-Pad2): track 0.00 -> 36.8 mm, vias 0 -> 2
- net /CPU/CPURST: track 0.00 -> 35.6 mm, vias 0 -> 2
- net Net-(R512-Pad1): track 6.17 -> 35.5 mm
- net Net-(C819-Pad1): track 0.00 -> 24.2 mm
- net Net-(R513-Pad1): track 7.81 -> 31.5 mm
- net Net-(T501-Pad6): track 0.00 -> 21.8 mm
- net /RX_chain/RX_CHAIN: track 0.00 -> 21.3 mm, vias 0 -> 2
- net Net-(C816-Pad1): track 0.00 -> 20.0 mm
- net /TX_chain/LO_I: track 0.00 -> 18.1 mm, vias 0 -> 2
- net Net-(P808-Pad6): track 0.00 -> 17.5 mm, vias 0 -> 1
- net Net-(C506-Pad1): track 0.00 -> 16.9 mm, vias 0 -> 1
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Other:
- board size 336.6 x 85.1 mm -> 76.2 x 76.2 mm
- rule pad_to_mask_clearance: 0.2 -> 0

Commit message: some minor advancements
Parts:
- D301, D302, D303, D304, R304: moved to F.Cu
- moved R304 54.2 mm to (144.9, 58.3)
- moved D304 45.5 mm to (145.8, 59.9), turned to 180 degrees
- moved D303 21.6 mm to (121.4, 69.8), turned to 90 degrees
- moved D301 6.86 mm to (100.1, 59.3), turned to 0 degrees
Routing:
- net GND: track 258.1 -> 261.6 mm, vias 22 -> 23
- net Net-(C311-Pad1): track 0.00 -> 3.46 mm, vias 0 -> 1
- net Net-(C506-Pad2): track 3.69 -> 4.21 mm, vias 0 -> 1
