File: hardware/rx_chain.sch (KiCad schematic (older format))
At the start: 23 parts, among them T601 TRANSFO2, U601 74LVC1G3157, U602 74LVC1G3157, U603 TL972IDR

Commit message: Linked first components to footprints and updated schematic plot
Parts:
- C601, C602, C603, C604, C605, C606, C607: footprint (none) -> Capacitors_SMD:C_0805
- R601, R602, R603, R604, R605, R606: footprint (none) -> Resistors_SMD:R_0805_HandSoldering
- U603: footprint (none) -> Housings_SOIC:SOIC-8_3.9x4.9mm_Pitch1.27mm
Changed lines of the file:
@@
 RX_CHAIN
 $Comp
-L GND #PWR601
+L GND #PWR040
 U 1 1 57E45141
 P 1600 3600
-F 0 "#PWR601" H 1600 3350 50  0001 C CNN
+F 0 "#PWR040" H 1600 3350 50  0001 C CNN
 F 1 "GND" H 1600 3450 50  0000 C CNN
 F 2 "" H 1600 3600 50  0000 C CNN
@@
 F 0 "T601" H 2200 3600 50  0000 C CNN
 F 1 "TRANSFO2" H 2200 2600 50  0000 C CNN
-F 2 "" H 2200 3100 50  0000 C CNN
+F 2 "" H 2200 3100 50  0001 C CNN
 F 3 "" H 2200 3100 50  0000 C CNN
 	1    2200 3100
@@
 $EndComp
 $Comp
-L GND #PWR603
+L GND #PWR041
 U 1 1 57E45302
 P 2800 3800
-F 0 "#PWR603" H 2800 3550 50  0001 C CNN
+F 0 "#PWR041" H 2800 3550 50  0001 C CNN
 F 1 "GND" H 2800 3650 50  0000 C CNN
 F 2 "" H 2800 3800 50  0000 C CNN
@@
 $EndComp
 $Comp
-L +Vlogic #PWR604
+L +Vlogic #PWR042
 U 1 1 57E45597
 P 4000 2550
-F 0 "#PWR604" H 4000 2350 50  0001 C CNN
+F 0 "#PWR042" H 4000 2350 50  0001 C CNN
 F 1 "+Vlogic" H 4000 2750 50  0000 C CNN
 F 2 "" H 4000 2550 50  0000 C CNN
@@
 F 0 "R601" V 4430 2900 50  0000 C CNN
 F 1 "100R" V 4350 2900 50  0000 C CNN
-F 2 "" V 4280 2900 50  0000 C CNN
+F 2 "Resistors_SMD:R_0805_HandSoldering" V 4280 2900 50  0001 C CNN
 F 3 "" H 4350 2900 50  0000 C CNN
 	1    4350 2900
@@
 F 0 "R602" V 4430 3900 50  0000 C CNN
 F 1 "100R" V 4350 3900 50  0000 C CNN
-F 2 "" V 4280 3900 50  0000 C CNN
+F 2 "Resistors_SMD:R_0805_HandSoldering" V 4280 3900 50  0001 C CNN
 F 3 "" H 4350 3900 50  0000 C CNN
 	1    4350 3900
@@
 F 0 "C602" H 4375 3300 50  0000 L CNN
 F 1 "C" H 4375 3100 50  0000 L CNN
-F 2 "" H 4388 3050 50  0000 C CNN
+F 2 "Capacitors_SMD:C_0805" H 4388 3050 50  0001 C CNN
 F 3 "" H 4350 3200 50  0000 C CNN
 	1    4350 3200
@@
 F 0 "C603" H 4375 4300 50  0000 L CNN
 F 1 "C" H 4375 4100 50  0000 L CNN
-F 2 "" H 4388 4050 50  0000 C CNN
+F 2 "Capacitors_SMD:C_0805" H 4388 4050 50  0001 C CNN
 F 3 "" H 4350 4200 50  0000 C CNN
 	1    4350 4200
@@
 F 0 "C605" H 5825 4100 50  0000 L CNN
 F 1 "C" H 5825 3900 50  0000 L CNN
-F 2 "" H 5838 3850 50  0000 C CNN
+F 2 "Capacitors_SMD:C_0805" H 5838 3850 50  0001 C CNN
 F 3 "" H 5800 4000 50  0000 C CNN
 	1    5800 4000
@@
 F 0 "C604" H 5825 3100 50  0000 L CNN
 F 1 "C" H 5825 2900 50  0000 L CNN
-F 2 "" H 5838 2850 50  0000 C CNN
+F 2 "Capacitors_SMD:C_0805" H 5838 2850 50  0001 C CNN
 F 3 "" H 5800 3000 50  0000 C CNN
 	1    5800 3000
@@
 F 0 "L601" V 4650 2650 50  0000 C CNN
 F 1 "440µH" V 4850 2650 50  0000 C CNN
-F 2 "" H 4750 2650 50  0000 C CNN
+F 2 "" H 4750 2650 50  0001 C CNN
 F 3 "" H 4750 2650 50  0000 C CNN
 	1    4750 2650
@@
 F 0 "L603" V 5300 2650 50  0000 C CNN
 F 1 "440µH" V 5500 2650 50  0000 C CNN
-F 2 "" H 5400 2650 50  0000 C CNN
+F 2 "" H 5400 2650 50  0001 C CNN
 F 3 "" H 5400 2650 50  0000 C CNN
 	1    5400 2650
@@
 F 0 "L602" V 4650 3650 50  0000 C CNN
 F 1 "440µH" V 4850 3650 50  0000 C CNN
-F 2 "" H 4750 3650 50  0000 C CNN
+F 2 "" H 4750 3650 50  0001 C CNN
 F 3 "" H 4750 3650 50  0000 C CNN
 	1    4750 3650
@@
 F 0 "L604" V 5300 3650 50  0000 C CNN
 F 1 "440µH" V 5500 3650 50  0000 C CNN
-F 2 "" H 5400 3650 50  0000 C CNN
+F 2 "" H 5400 3650 50  0001 C CNN
 F 3 "" H 5400 3650 50  0000 C CNN
 	1    5400 3650
@@
 F 0 "U603" H 7500 3150 60  0000 C CNN
 F 1 "TL972IDR" H 7500 3750 60  0000 C CNN
-F 2 "" H 7550 3450 60  0001 C CNN
+F 2 "Housings_SOIC:SOIC-8_3.9x4.9mm_Pitch1.27mm" H 7550 3450 60  0001 C CNN
 F 3 "" H 7550 3450 60  0001 C CNN
 	1    7500 3450
@@
 $EndComp
 $Comp
-L +Vlogic #PWR606
+L +Vlogic #PWR043
 U 1 1 57E48734
 P 8000 3250
-F 0 "#PWR606" H 8000 3050 50  0001 C CNN
+F 0 "#PWR043" H 8000 3050 50  0001 C CNN
 F 1 "+Vlogic" H 8000 3450 50  0000 C CNN
 F 2 "" H 8000 3250 50  0000 C CNN
@@
 F 0 "R603" V 6230 2900 50  0000 C CNN
 F 1 "100R" V 6150 2900 50  0000 C CNN
-F 2 "" V 6080 2900 50  0000 C CNN
+F 2 "Resistors_SMD:R_0805_HandSoldering" V 6080 2900 50  0001 C CNN
 F 3 "" H 6150 2900 50  0000 C CNN
 	1    6150 2900
@@
 $EndComp
 $Comp
-L GND #PWR605
+L GND #PWR044
 U 1 1 57E4894A
 P 7000 3700
-F 0 "#PWR605" H 7000 3450 50  0001 C CNN
+F 0 "#PWR044" H 7000 3450 50  0001 C CNN
 F 1 "GND" H 7000 3550 50  0000 C CNN
 F 2 "" H 7000 3700 50  0000 C CNN
@@
 F 0 "D602" H 1600 3400 50  0000 C CNN
 F 1 "ZENER" H 1600 3200 50  0000 C CNN
-F 2 "" H 1600 3300 50  0000 C CNN
+F 2 "" H 1600 3300 50  0001 C CNN
 F 3 "" H 1600 3300 50  0000 C CNN
 	1    1600 3300
@@
 F 0 "D601" H 1600 3000 50  0000 C CNN
 F 1 "ZENER" H 1600 2800 50  0000 C CNN
-F 2 "" H 1600 2900 50  0000 C CNN
+F 2 "" H 1600 2900 50  0001 C CNN
 F 3 "" H 1600 2900 50  0000 C CNN
 	1    1600 2900
@@
 F 0 "R604" V 6330 3850 50  0000 C CNN
 F 1 "100R" V 6250 3850 50  0000 C CNN
-F 2 "" V 6180 3850 50  0000 C CNN
+F 2 "Resistors_SMD:R_0805_HandSoldering" V 6180 3850 50  0001 C CNN
 F 3 "" H 6250 3850 50  0000 C CNN
 	1    6250 3850
@@
 F 0 "C601" H 2425 4000 50  0000 L CNN
 F 1 "100nF" H 2425 3800 50  0000 L CNN
-F 2 "" H 2438 3750 50  0000 C CNN
+F 2 "Capacitors_SMD:C_0805" H 2438 3750 50  0001 C CNN
 F 3 "" H 2400 3900 50  0000 C CNN
 	1    2400 3900
@@
 $EndComp
 $Comp
-L GND #PWR602
+L GND #PWR045
 U 1 1 57EAE15A
 P 2400 4100
-F 0 "#PWR602" H 2400 3850 50  0001 C CNN
+F 0 "#PWR045" H 2400 3850 50  0001 C CNN
 F 1 "GND" H 2400 3950 50  0000 C CNN
 F 2 "" H 2400 4100 50  0000 C CNN
@@
 F 0 "C606" H 6675 3200 50  0000 L CNN
 F 1 "100pF" H 6675 3000 50  0000 L CNN
-F 2 "" H 6688 2950 50  0000 C CNN
+F 2 "Capacitors_SMD:C_0805" H 6688 2950 50  0001 C CNN
 F 3 "" H 6650 3100 50  0000 C CNN
 	1    6650 3100
@@
 F 0 "C607" H 8575 3850 50  0000 L CNN
 F 1 "100pF" H 8575 3650 50  0000 L CNN
-F 2 "" H 8588 3600 50  0000 C CNN
+F 2 "Capacitors_SMD:C_0805" H 8588 3600 50  0001 C CNN
 F 3 "" H 8550 3750 50  0000 C CNN
 	1    8550 3750
@@
 F 0 "R605" V 6930 3100 50  0000 C CNN
 F 1 "33k" V 6850 3100 50  0000 C CNN
-F 2 "" V 6780 3100 50  0000 C CNN
+F 2 "Resistors_SMD:R_0805_HandSoldering" V 6780 3100 50  0001 C CNN
 F 3 "" H 6850 3100 50  0000 C CNN
 	1    6850 3100
@@
 F 0 "R606" V 8380 3750 50  0000 C CNN
 F 1 "33k" V 8300 3750 50  0000 C CNN
-F 2 "" V 8230 3750 50  0000 C CNN
+F 2 "Resistors_SMD:R_0805_HandSoldering" V 8230 3750 50  0001 C CNN
 F 3 "" H 8300 3750 50  0000 C CNN
 	1    8300 3750

Commit message: Changed SWR microstrip for two transformers and gave missing values for components
Parts:
- removed D601, D602: ZENER, symbol ZENER
- added D601, D602: BAP65-02, symbol D
- C602, C603, C604, C605: value C -> 68nF
- L601, L602, L603, L604: value 440µH -> 470µH
Connections:
- net GND: now also D602.2 (A)
- net RX_CHAIN: now also D601.2 (A)
- new net: D601.1 (K), D602.1 (K)
Changed lines of the file:
@@
 RX_CHAIN
 $Comp
-L GND #PWR040
+L GND #PWR601
 U 1 1 57E45141
 P 1600 3600
-F 0 "#PWR040" H 1600 3350 50  0001 C CNN
+F 0 "#PWR601" H 1600 3350 50  0001 C CNN
 F 1 "GND" H 1600 3450 50  0000 C CNN
 F 2 "" H 1600 3600 50  0000 C CNN
@@
 $EndComp
 $Comp
-L GND #PWR041
+L GND #PWR603
 U 1 1 57E45302
 P 2800 3800
-F 0 "#PWR041" H 2800 3550 50  0001 C CNN
+F 0 "#PWR603" H 2800 3550 50  0001 C CNN
 F 1 "GND" H 2800 3650 50  0000 C CNN
 F 2 "" H 2800 3800 50  0000 C CNN
@@
 $EndComp
 $Comp
-L +Vlogic #PWR042
+L +Vlogic #PWR604
 U 1 1 57E45597
 P 4000 2550
-F 0 "#PWR042" H 4000 2350 50  0001 C CNN
+F 0 "#PWR604" H 4000 2350 50  0001 C CNN
 F 1 "+Vlogic" H 4000 2750 50  0000 C CNN
 F 2 "" H 4000 2550 50  0000 C CNN
@@
 P 4350 3200
 F 0 "C602" H 4375 3300 50  0000 L CNN
-F 1 "C" H 4375 3100 50  0000 L CNN
+F 1 "68nF" H 4375 3100 50  0000 L CNN
 F 2 "Capacitors_SMD:C_0805" H 4388 3050 50  0001 C CNN
 F 3 "" H 4350 3200 50  0000 C CNN
@@
 P 4350 4200
 F 0 "C603" H 4375 4300 50  0000 L CNN
-F 1 "C" H 4375 4100 50  0000 L CNN
+F 1 "68nF" H 4375 4100 50  0000 L CNN
 F 2 "Capacitors_SMD:C_0805" H 4388 4050 50  0001 C CNN
 F 3 "" H 4350 4200 50  0000 C CNN
@@
 P 5800 4000
 F 0 "C605" H 5825 4100 50  0000 L CNN
-F 1 "C" H 5825 3900 50  0000 L CNN
+F 1 "68nF" H 5825 3900 50  0000 L CNN
 F 2 "Capacitors_SMD:C_0805" H 5838 3850 50  0001 C CNN
 F 3 "" H 5800 4000 50  0000 C CNN
@@
 P 5800 3000
 F 0 "C604" H 5825 3100 50  0000 L CNN
-F 1 "C" H 5825 2900 50  0000 L CNN
+F 1 "68nF" H 5825 2900 50  0000 L CNN
 F 2 "Capacitors_SMD:C_0805" H 5838 2850 50  0001 C CNN
 F 3 "" H 5800 3000 50  0000 C CNN
@@
 P 4750 2650
 F 0 "L601" V 4650 2650 50  0000 C CNN
-F 1 "440µH" V 4850 2650 50  0000 C CNN
+F 1 "470µH" V 4850 2650 50  0000 C CNN
 F 2 "" H 4750 2650 50  0001 C CNN
 F 3 "" H 4750 2650 50  0000 C CNN
@@
 P 5400 2650
 F 0 "L603" V 5300 2650 50  0000 C CNN
-F 1 "440µH" V 5500 2650 50  0000 C CNN
+F 1 "470µH" V 5500 2650 50  0000 C CNN
 F 2 "" H 5400 2650 50  0001 C CNN
 F 3 "" H 5400 2650 50  0000 C CNN
@@
 P 4750 3650
 F 0 "L602" V 4650 3650 50  0000 C CNN
-F 1 "440µH" V 4850 3650 50  0000 C CNN
+F 1 "470µH" V 4850 3650 50  0000 C CNN
 F 2 "" H 4750 3650 50  0001 C CNN
 F 3 "" H 4750 3650 50  0000 C CNN
@@
 P 5400 3650
 F 0 "L604" V 5300 3650 50  0000 C CNN
-F 1 "440µH" V 5500 3650 50  0000 C CNN
+F 1 "470µH" V 5500 3650 50  0000 C CNN
 F 2 "" H 5400 3650 50  0001 C CNN
 F 3 "" H 5400 3650 50  0000 C CNN
@@
 $EndComp
 $Comp
-L +Vlogic #PWR043
+L +Vlogic #PWR606
 U 1 1 57E48734
 P 8000 3250
-F 0 "#PWR043" H 8000 3050 50  0001 C CNN
+F 0 "#PWR606" H 8000 3050 50  0001 C CNN
 F 1 "+Vlogic" H 8000 3450 50  0000 C CNN
 F 2 "" H 8000 3250 50  0000 C CNN
@@
 $EndComp
 $Comp
-L GND #PWR044
+L GND #PWR605
 U 1 1 57E4894A
 P 7000 3700
-F 0 "#PWR044" H 7000 3450 50  0001 C CNN
+F 0 "#PWR605" H 7000 3450 50  0001 C CNN
 F 1 "GND" H 7000 3550 50  0000 C CNN
 F 2 "" H 7000 3700 50  0000 C CNN
@@
 	1800 3600 1600 3600
 Wire Wire Line
-	1600 2600 1600 2700
+	1600 2600 1600 2750
 Wire Wire Line
 	2600 3000 2600 3200
@@
 Connection ~ 4150 4350
 Connection ~ 4350 3350
-$Comp
-L ZENER D602
-U 1 1 57ED018F
-P 1600 3300
-F 0 "D602" H 1600 3400 50  0000 C CNN
-F 1 "ZENER" H 1600 3200 50  0000 C CNN
-F 2 "" H 1600 3300 50  0001 C CNN
-F 3 "" H 1600 3300 50  0000 C CNN
-	1    1600 3300
-	0    1    1    0
-$EndComp
-$Comp
-L ZENER D601
-U 1 1 57ED027D
-P 1600 2900
-F 0 "D601" H 1600 3000 50  0000 C CNN
-F 1 "ZENER" H 1600 2800 50  0000 C CNN
-F 2 "" H 1600 2900 50  0001 C CNN
-F 3 "" H 1600 2900 50  0000 C CNN
-	1    1600 2900
-	0    -1   -1   0
-$EndComp
-Wire Wire Line
-	1600 3600 1600 3500
+Wire Wire Line
+	1600 3600 1600 3450
 Wire Wire Line
 	1800 2600 1800 2900
@@
 $EndComp
 $Comp
-L GND #PWR045
+L GND #PWR602
 U 1 1 57EAE15A
 P 2400 4100
-F 0 "#PWR045" H 2400 3850 50  0001 C CNN
+F 0 "#PWR602" H 2400 3850 50  0001 C CNN
 F 1 "GND" H 2400 3950 50  0000 C CNN
 F 2 "" H 2400 4100 50  0000 C CNN
@@
 Wire Wire Line
 	6250 3650 6250 3700
+$Comp
+L D D602
+U 1 1 57F0CC22
+P 1600 3300
+F 0 "D602" H 1600 3400 50  0000 C CNN
+F 1 "BAP65-02" H 1600 3200 50  0000 C CNN
+F 2 "" H 1600 3300 50  0000 C CNN
+F 3 "" H 1600 3300 50  0000 C CNN
+	1    1600 3300
+	0    1    1    0
+$EndComp
+$Comp
+L D D601
+U 1 1 57F0CC85
+P 1600 2900
+F 0 "D601" H 1600 3000 50  0000 C CNN
+F 1 "BAP65-02" H 1600 2800 50  0000 C CNN
+F 2 "" H 1600 2900 50  0000 C CNN
+F 3 "" H 1600 2900 50  0000 C CNN
+	1    1600 2900
+	0    -1   -1   0
+$EndComp
+Wire Wire Line
+	1600 3050 1600 3150
 $EndSCHEMATC

Commit message: Fixed some bugs and annotated rest of the footprints
Parts:
- C601, C602, C603, C604, C605, C606, C607: footprint Capacitors_SMD:C_0805 -> Capacitors_SMD:C_0805_HandSoldering
- D601, D602: footprint (none) -> Diodes_SMD:SOD-523
- L601, L602, L603, L604: footprint (none) -> dodekaedri:SMT_1007
- T601: footprint (none) -> dodekaedri:transf_5_pin
- U601, U602: footprint (none) -> TO_SOT_Packages_SMD:SOT-23-6_Handsoldering
Changed lines of the file:
@@
 RX_CHAIN
 $Comp
-L GND #PWR601
+L GND #PWR038
 U 1 1 57E45141
 P 1600 3600
-F 0 "#PWR601" H 1600 3350 50  0001 C CNN
+F 0 "#PWR038" H 1600 3350 50  0001 C CNN
 F 1 "GND" H 1600 3450 50  0000 C CNN
 F 2 "" H 1600 3600 50  0000 C CNN
@@
 F 0 "T601" H 2200 3600 50  0000 C CNN
 F 1 "TRANSFO2" H 2200 2600 50  0000 C CNN
-F 2 "" H 2200 3100 50  0001 C CNN
+F 2 "dodekaedri:transf_5_pin" H 2200 3100 50  0001 C CNN
 F 3 "" H 2200 3100 50  0000 C CNN
 	1    2200 3100
@@
 F 0 "U601" H 3350 2550 60  0000 C CNN
 F 1 "74LVC1G3157" H 3350 3050 60  0000 C CNN
-F 2 "" H 3350 2700 60  0001 C CNN
+F 2 "TO_SOT_Packages_SMD:SOT-23-6_Handsoldering" H 3350 2700 60  0001 C CNN
 F 3 "" H 3350 2700 60  0001 C CNN
 	1    3350 2800
@@
 F 0 "U602" H 3350 3150 60  0000 C CNN
 F 1 "74LVC1G3157" H 3350 3650 60  0000 C CNN
-F 2 "" H 3350 3300 60  0001 C CNN
+F 2 "TO_SOT_Packages_SMD:SOT-23-6_Handsoldering" H 3350 3300 60  0001 C CNN
 F 3 "" H 3350 3300 60  0001 C CNN
 	1    3350 3400
@@
 $EndComp
 $Comp
-L GND #PWR603
+L GND #PWR039
 U 1 1 57E45302
 P 2800 3800
-F 0 "#PWR603" H 2800 3550 50  0001 C CNN
+F 0 "#PWR039" H 2800 3550 50  0001 C CNN
 F 1 "GND" H 2800 3650 50  0000 C CNN
 F 2 "" H 2800 3800 50  0000 C CNN
@@
 $EndComp
 $Comp
-L +Vlogic #PWR604
+L +Vlogic #PWR040
 U 1 1 57E45597
 P 4000 2550
-F 0 "#PWR604" H 4000 2350 50  0001 C CNN
+F 0 "#PWR040" H 4000 2350 50  0001 C CNN
 F 1 "+Vlogic" H 4000 2750 50  0000 C CNN
 F 2 "" H 4000 2550 50  0000 C CNN
@@
 F 0 "C602" H 4375 3300 50  0000 L CNN
 F 1 "68nF" H 4375 3100 50  0000 L CNN
-F 2 "Capacitors_SMD:C_0805" H 4388 3050 50  0001 C CNN
+F 2 "Capacitors_SMD:C_0805_HandSoldering" H 4388 3050 50  0001 C CNN
 F 3 "" H 4350 3200 50  0000 C CNN
 	1    4350 3200
@@
 F 0 "C603" H 4375 4300 50  0000 L CNN
 F 1 "68nF" H 4375 4100 50  0000 L CNN
-F 2 "Capacitors_SMD:C_0805" H 4388 4050 50  0001 C CNN
+F 2 "Capacitors_SMD:C_0805_HandSoldering" H 4388 4050 50  0001 C CNN
 F 3 "" H 4350 4200 50  0000 C CNN
 	1    4350 4200
@@
 F 0 "C605" H 5825 4100 50  0000 L CNN
 F 1 "68nF" H 5825 3900 50  0000 L CNN
-F 2 "Capacitors_SMD:C_0805" H 5838 3850 50  0001 C CNN
+F 2 "Capacitors_SMD:C_0805_HandSoldering" H 5838 3850 50  0001 C CNN
 F 3 "" H 5800 4000 50  0000 C CNN
 	1    5800 4000
@@
 F 0 "C604" H 5825 3100 50  0000 L CNN
 F 1 "68nF" H 5825 2900 50  0000 L CNN
-F 2 "Capacitors_SMD:C_0805" H 5838 2850 50  0001 C CNN
+F 2 "Capacitors_SMD:C_0805_HandSoldering" H 5838 2850 50  0001 C CNN
 F 3 "" H 5800 3000 50  0000 C CNN
 	1    5800 3000
@@
 F 0 "L601" V 4650 2650 50  0000 C CNN
 F 1 "470µH" V 4850 2650 50  0000 C CNN
-F 2 "" H 4750 2650 50  0001 C CNN
+F 2 "dodekaedri:SMT_1007" H 4750 2650 50  0001 C CNN
 F 3 "" H 4750 2650 50  0000 C CNN
 	1    4750 2650
@@
 F 0 "L603" V 5300 2650 50  0000 C CNN
 F 1 "470µH" V 5500 2650 50  0000 C CNN
-F 2 "" H 5400 2650 50  0001 C CNN
+F 2 "dodekaedri:SMT_1007" H 5400 2650 50  0001 C CNN
 F 3 "" H 5400 2650 50  0000 C CNN
 	1    5400 2650
@@
 F 0 "L602" V 4650 3650 50  0000 C CNN
 F 1 "470µH" V 4850 3650 50  0000 C CNN
-F 2 "" H 4750 3650 50  0001 C CNN
+F 2 "dodekaedri:SMT_1007" H 4750 3650 50  0001 C CNN
 F 3 "" H 4750 3650 50  0000 C CNN
 	1    4750 3650
@@
 F 0 "L604" V 5300 3650 50  0000 C CNN
 F 1 "470µH" V 5500 3650 50  0000 C CNN
-F 2 "" H 5400 3650 50  0001 C CNN
+F 2 "dodekaedri:SMT_1007" H 5400 3650 50  0001 C CNN
 F 3 "" H 5400 3650 50  0000 C CNN
 	1    5400 3650
@@
 $EndComp
 $Comp
-L +Vlogic #PWR606
+L +Vlogic #PWR041
 U 1 1 57E48734
 P 8000 3250
-F 0 "#PWR606" H 8000 3050 50  0001 C CNN
+F 0 "#PWR041" H 8000 3050 50  0001 C CNN
 F 1 "+Vlogic" H 8000 3450 50  0000 C CNN
 F 2 "" H 8000 3250 50  0000 C CNN
@@
 $EndComp
 $Comp
-L GND #PWR605
+L GND #PWR042
 U 1 1 57E4894A
 P 7000 3700
-F 0 "#PWR605" H 7000 3450 50  0001 C CNN
+F 0 "#PWR042" H 7000 3450 50  0001 C CNN
 F 1 "GND" H 7000 3550 50  0000 C CNN
 F 2 "" H 7000 3700 50  0000 C CNN
@@
 F 0 "C601" H 2425 4000 50  0000 L CNN
 F 1 "100nF" H 2425 3800 50  0000 L CNN
-F 2 "Capacitors_SMD:C_0805" H 2438 3750 50  0001 C CNN
+F 2 "Capacitors_SMD:C_0805_HandSoldering" H 2438 3750 50  0001 C CNN
 F 3 "" H 2400 3900 50  0000 C CNN
 	1    2400 3900
@@
 $EndComp
 $Comp
-L GND #PWR602
+L GND #PWR043
 U 1 1 57EAE15A
 P 2400 4100
-F 0 "#PWR602" H 2400 3850 50  0001 C CNN
+F 0 "#PWR043" H 2400 3850 50  0001 C CNN
 F 1 "GND" H 2400 3950 50  0000 C CNN
 F 2 "" H 2400 4100 50  0000 C CNN
@@
 F 0 "C606" H 6675 3200 50  0000 L CNN
 F 1 "100pF" H 6675 3000 50  0000 L CNN
-F 2 "Capacitors_SMD:C_0805" H 6688 2950 50  0001 C CNN
+F 2 "Capacitors_SMD:C_0805_HandSoldering" H 6688 2950 50  0001 C CNN
 F 3 "" H 6650 3100 50  0000 C CNN
 	1    6650 3100
@@
 F 0 "C607" H 8575 3850 50  0000 L CNN
 F 1 "100pF" H 8575 3650 50  0000 L CNN
-F 2 "Capacitors_SMD:C_0805" H 8588 3600 50  0001 C CNN
+F 2 "Capacitors_SMD:C_0805_HandSoldering" H 8588 3600 50  0001 C CNN
 F 3 "" H 8550 3750 50  0000 C CNN
 	1    8550 3750
@@
 F 0 "D602" H 1600 3400 50  0000 C CNN
 F 1 "BAP65-02" H 1600 3200 50  0000 C CNN
-F 2 "" H 1600 3300 50  0000 C CNN
+F 2 "Diodes_SMD:SOD-523" H 1600 3300 50  0001 C CNN
 F 3 "" H 1600 3300 50  0000 C CNN
 	1    1600 3300
@@
 F 0 "D601" H 1600 3000 50  0000 C CNN
 F 1 "BAP65-02" H 1600 2800 50  0000 C CNN
-F 2 "" H 1600 2900 50  0000 C CNN
+F 2 "Diodes_SMD:SOD-523" H 1600 2900 50  0001 C CNN
 F 3 "" H 1600 2900 50  0000 C CNN
 	1    1600 2900

Commit message: halfway through layout
Parts:
- removed D601, D602: BAP65-02, Diodes_SMD:SOD-523, symbol D
- added C608: 100nF, Capacitors_SMD:C_0805_HandSoldering, symbol C
- C606, C607: value 100pF -> 1nF
- R605, R606: value 33k -> 1k
Connections:
- net RX_BIAS: now also C608.2
- net at L602.1, R602.1, U602.4 (A): now also C608.1
Other:
- note added: "R605 and R606:\n10k and 100pF\nfor more gain"
Changed lines of the file:
@@
 Comment4 ""
 $EndDescr
-Text HLabel 1300 2600 0    60   Input ~ 0
+Text HLabel 1650 2600 0    60   Input ~ 0
 RX_CHAIN
 $Comp
 L GND #PWR040
 U 1 1 57E45141
-P 1600 3600
-F 0 "#PWR040" H 1600 3350 50  0001 C CNN
-F 1 "GND" H 1600 3450 50  0000 C CNN
-F 2 "" H 1600 3600 50  0000 C CNN
-F 3 "" H 1600 3600 50  0000 C CNN
-	1    1600 3600
+P 1800 3600
+F 0 "#PWR040" H 1800 3350 50  0001 C CNN
+F 1 "GND" H 1800 3450 50  0000 C CNN
+F 2 "" H 1800 3600 50  0000 C CNN
+F 3 "" H 1800 3600 50  0000 C CNN
+	1    1800 3600
 	1    0    0    -1
 $EndComp
@@
 	1800 3300 1800 3600
 Wire Wire Line
-	1800 3600 1600 3600
-Wire Wire Line
-	1600 2600 1600 2750
-Wire Wire Line
 	2600 3000 2600 3200
 Wire Wire Line
@@
 Connection ~ 4350 3350
 Wire Wire Line
-	1600 3600 1600 3450
-Wire Wire Line
 	1800 2600 1800 2900
 Wire Wire Line
-	1300 2600 1800 2600
-Connection ~ 1600 2600
+	1650 2600 1800 2600
 $Comp
 L R R604
@@
 P 6650 3100
 F 0 "C606" H 6675 3200 50  0000 L CNN
-F 1 "100pF" H 6675 3000 50  0000 L CNN
+F 1 "1nF" H 6675 3000 50  0000 L CNN
 F 2 "Capacitors_SMD:C_0805_HandSoldering" H 6688 2950 50  0001 C CNN
 F 3 "" H 6650 3100 50  0000 C CNN
@@
 P 8550 3750
 F 0 "C607" H 8575 3850 50  0000 L CNN
-F 1 "100pF" H 8575 3650 50  0000 L CNN
+F 1 "1nF" H 8575 3650 50  0000 L CNN
 F 2 "Capacitors_SMD:C_0805_HandSoldering" H 8588 3600 50  0001 C CNN
 F 3 "" H 8550 3750 50  0000 C CNN
@@
 P 6850 3100
 F 0 "R605" V 6930 3100 50  0000 C CNN
-F 1 "33k" V 6850 3100 50  0000 C CNN
+F 1 "1k" V 6850 3100 50  0000 C CNN
 F 2 "Resistors_SMD:R_0805_HandSoldering" V 6780 3100 50  0001 C CNN
 F 3 "" H 6850 3100 50  0000 C CNN
@@
 P 8300 3750
 F 0 "R606" V 8380 3750 50  0000 C CNN
-F 1 "33k" V 8300 3750 50  0000 C CNN
+F 1 "1k" V 8300 3750 50  0000 C CNN
 F 2 "Resistors_SMD:R_0805_HandSoldering" V 8230 3750 50  0001 C CNN
 F 3 "" H 8300 3750 50  0000 C CNN
@@
 	6250 3650 6250 3700
 $Comp
-L D D602
-U 1 1 57F0CC22
-P 1600 3300
-F 0 "D602" H 1600 3400 50  0000 C CNN
-F 1 "BAP65-02" H 1600 3200 50  0000 C CNN
-F 2 "Diodes_SMD:SOD-523" H 1600 3300 50  0001 C CNN
-F 3 "" H 1600 3300 50  0000 C CNN
-	1    1600 3300
-	0    1    1    0
-$EndComp
-$Comp
-L D D601
-U 1 1 57F0CC85
-P 1600 2900
-F 0 "D601" H 1600 3000 50  0000 C CNN
-F 1 "BAP65-02" H 1600 2800 50  0000 C CNN
-F 2 "Diodes_SMD:SOD-523" H 1600 2900 50  0001 C CNN
-F 3 "" H 1600 2900 50  0000 C CNN
-	1    1600 2900
-	0    -1   -1   0
-$EndComp
-Wire Wire Line
-	1600 3050 1600 3150
+L C C608
+U 1 1 57F2AC7C
+P 3850 3900
+F 0 "C608" H 3875 4000 50  0000 L CNN
+F 1 "100nF" H 3875 3800 50  0000 L CNN
+F 2 "Capacitors_SMD:C_0805_HandSoldering" H 3888 3750 50  0001 C CNN
+F 3 "" H 3850 3900 50  0000 C CNN
+	1    3850 3900
+	1    0    0    -1
+$EndComp
+Wire Wire Line
+	3850 3500 3850 3750
+Connection ~ 3850 3500
+Wire Wire Line
+	3850 4050 3850 4350
+Connection ~ 3850 4350
+Text Notes 8150 4250 0    60   ~ 0
+R605 and R606:\n10k and 100pF\nfor more gain
 $EndSCHEMATC

Commit message: fixed serious schematic and thus layout bug
Connections:
- net +Vlogic: now also C608.1
- net at L602.1, R602.1, U602.4 (A): no longer C608.1
Changed lines of the file:
@@
 	4350 2650 4450 2650
-Wire Wire Line
-	3750 3500 4000 3500
-Wire Wire Line
-	4000 3500 4000 3650
-Connection ~ 4350 3650
 Wire Wire Line
 	3750 2900 4150 2900
@@
 RX_BIAS
 Wire Wire Line
-	6050 3500 6050 3350
+	6050 3350 6050 3500
 Wire Wire Line
-	6050 3350 4150 3350
+	4150 3350 6050 3350
 Connection ~ 5800 3350
 Wire Wire Line
@@
 $EndComp
 Wire Wire Line
-	3850 3500 3850 3750
-Connection ~ 3850 3500
-Wire Wire Line
 	3850 4050 3850 4350
 Connection ~ 3850 4350
 Text Notes 8150 4250 0    60   ~ 0
 R605 and R606:\n10k and 100pF\nfor more gain
+Connection ~ 4350 3650
+Wire Wire Line
+	4000 3500 4000 3650
+Wire Wire Line
+	3750 3500 4000 3500
+Wire Wire Line
+	3850 3750 3850 3400
+Connection ~ 3850 3400
 $EndSCHEMATC

Commit message: changed some component values
Changed lines of the file:
@@
 RX_BIAS
 Wire Wire Line
-	6050 3350 6050 3500
+	6050 3500 6050 3350
 Wire Wire Line
-	4150 3350 6050 3350
+	6050 3350 4150 3350
 Connection ~ 5800 3350
 Wire Wire Line
