File: hardware/freq_synth.sch (KiCad schematic (older format))
At the start: 15 parts, among them U201 MIC5365, U202 SI5351A

Commit message: Linked first components to footprints and updated schematic plot
Parts:
- C201, C202, C203, C204, C205: footprint (none) -> Capacitors_SMD:C_0805
- R201, R202, R203, R204, R205, R206, R207: footprint (none) -> Resistors_SMD:R_0805_HandSoldering
Changed lines of the file:
@@
 F 0 "R207" H 7830 4520 50  0000 L CNN
 F 1 "50R" H 7830 4460 50  0000 L CNN
-F 2 "" H 7800 4500 50  0000 C CNN
+F 2 "Resistors_SMD:R_0805_HandSoldering" H 7800 4500 50  0001 C CNN
 F 3 "" H 7800 4500 50  0000 C CNN
 	1    7800 4500
@@
 F 0 "R205" H 7630 3920 50  0000 L CNN
 F 1 "50R" H 7630 3860 50  0000 L CNN
-F 2 "" H 7600 3900 50  0000 C CNN
+F 2 "Resistors_SMD:R_0805_HandSoldering" H 7600 3900 50  0001 C CNN
 F 3 "" H 7600 3900 50  0000 C CNN
 	1    7600 3900
@@
 F 0 "R206" H 7830 3920 50  0000 L CNN
 F 1 "50R" H 7830 3860 50  0000 L CNN
-F 2 "" H 7800 3900 50  0000 C CNN
+F 2 "Resistors_SMD:R_0805_HandSoldering" H 7800 3900 50  0001 C CNN
 F 3 "" H 7800 3900 50  0000 C CNN
 	1    7800 3900
@@
 1,8Vrail
 $Comp
-L +Vlogic #PWR202
+L +Vlogic #PWR05
 U 1 1 57E31A13
 P 4350 2850
-F 0 "#PWR202" H 4350 2650 50  0001 C CNN
+F 0 "#PWR05" H 4350 2650 50  0001 C CNN
 F 1 "+Vlogic" H 4350 3050 50  0000 C CNN
 F 2 "" H 4350 2850 50  0000 C CNN
@@
 F 0 "C202" H 5110 3620 50  0000 L CNN
 F 1 "1µF" H 5110 3470 50  0000 L CNN
-F 2 "" H 5100 3550 50  0000 C CNN
+F 2 "Capacitors_SMD:C_0805" H 5100 3550 50  0001 C CNN
 F 3 "" H 5100 3550 50  0000 C CNN
 	1    5100 3550
@@
 F 0 "C201" H 4360 3220 50  0000 L CNN
 F 1 "1µF" H 4360 3070 50  0000 L CNN
-F 2 "" H 4350 3150 50  0000 C CNN
+F 2 "Capacitors_SMD:C_0805" H 4350 3150 50  0001 C CNN
 F 3 "" H 4350 3150 50  0000 C CNN
 	1    4350 3150
@@
 $EndComp
 $Comp
-L GND #PWR203
+L GND #PWR06
 U 1 1 57E31A2E
 P 4350 4200
-F 0 "#PWR203" H 4350 3950 50  0001 C CNN
+F 0 "#PWR06" H 4350 3950 50  0001 C CNN
 F 1 "GND" H 4350 4050 50  0000 C CNN
 F 2 "" H 4350 4200 50  0000 C CNN
@@
 $EndComp
 $Comp
-L +Vlogic #PWR201
+L +Vlogic #PWR07
 U 1 1 57E31A3B
 P 3750 3950
-F 0 "#PWR201" H 3750 3750 50  0001 C CNN
+F 0 "#PWR07" H 3750 3750 50  0001 C CNN
 F 1 "+Vlogic" H 3750 4150 50  0000 C CNN
 F 2 "" H 3750 3950 50  0000 C CNN
@@
 $EndComp
 $Comp
-L +Vlogic #PWR207
+L +Vlogic #PWR08
 U 1 1 57E31A41
 P 8050 3950
-F 0 "#PWR207" H 8050 3750 50  0001 C CNN
+F 0 "#PWR08" H 8050 3750 50  0001 C CNN
 F 1 "+Vlogic" H 8050 4150 50  0000 C CNN
 F 2 "" H 8050 3950 50  0000 C CNN
@@
 F 0 "R201" V 3680 4100 50  0000 C CNN
 F 1 "10k" V 3600 4100 50  0000 C CNN
-F 2 "" V 3530 4100 50  0000 C CNN
+F 2 "Resistors_SMD:R_0805_HandSoldering" V 3530 4100 50  0001 C CNN
 F 3 "" H 3600 4100 50  0000 C CNN
 	1    3600 4100
@@
 F 0 "R202" V 3980 4100 50  0000 C CNN
 F 1 "10k" V 3900 4100 50  0000 C CNN
-F 2 "" V 3830 4100 50  0000 C CNN
+F 2 "Resistors_SMD:R_0805_HandSoldering" V 3830 4100 50  0001 C CNN
 F 3 "" H 3900 4100 50  0000 C CNN
 	1    3900 4100
@@
 F 0 "C203" H 5710 4270 50  0000 L CNN
 F 1 "C_Small" H 5710 4120 50  0000 L CNN
-F 2 "" H 5700 4200 50  0000 C CNN
+F 2 "Capacitors_SMD:C_0805" H 5700 4200 50  0001 C CNN
 F 3 "" H 5700 4200 50  0000 C CNN
 	1    5700 4200
@@
 $EndComp
 $Comp
-L +Vlogic #PWR206
+L +Vlogic #PWR09
 U 1 1 57E31A5D
 P 6050 3550
-F 0 "#PWR206" H 6050 3350 50  0001 C CNN
+F 0 "#PWR09" H 6050 3350 50  0001 C CNN
 F 1 "+Vlogic" H 6050 3750 50  0000 C CNN
 F 2 "" H 6050 3550 50  0000 C CNN
@@
 F 0 "C205" H 8060 4170 50  0000 L CNN
 F 1 "100nF" H 8060 4020 50  0000 L CNN
-F 2 "" H 8050 4100 50  0000 C CNN
+F 2 "Capacitors_SMD:C_0805" H 8050 4100 50  0001 C CNN
 F 3 "" H 8050 4100 50  0000 C CNN
 	1    8050 4100
@@
 F 0 "C204" H 5910 3870 50  0000 L CNN
 F 1 "100nF" H 5910 3720 50  0000 L CNN
-F 2 "" H 5900 3800 50  0000 C CNN
+F 2 "Capacitors_SMD:C_0805" H 5900 3800 50  0001 C CNN
 F 3 "" H 5900 3800 50  0000 C CNN
 	1    5900 3800
@@
 $EndComp
 $Comp
-L GND #PWR205
+L GND #PWR010
 U 1 1 57E31A71
 P 5900 3950
-F 0 "#PWR205" H 5900 3700 50  0001 C CNN
+F 0 "#PWR010" H 5900 3700 50  0001 C CNN
 F 1 "GND" H 5900 3800 50  0000 C CNN
 F 2 "" H 5900 3950 50  0000 C CNN
@@
 $EndComp
 $Comp
-L GND #PWR208
+L GND #PWR011
 U 1 1 57E31A77
 P 8050 4200
-F 0 "#PWR208" H 8050 3950 50  0001 C CNN
+F 0 "#PWR011" H 8050 3950 50  0001 C CNN
 F 1 "GND" H 8050 4050 50  0000 C CNN
 F 2 "" H 8050 4200 50  0000 C CNN
@@
 F 0 "R204" H 7430 3920 50  0000 L CNN
 F 1 "50R" H 7430 3860 50  0000 L CNN
-F 2 "" H 7400 3900 50  0000 C CNN
+F 2 "Resistors_SMD:R_0805_HandSoldering" H 7400 3900 50  0001 C CNN
 F 3 "" H 7400 3900 50  0000 C CNN
 	1    7400 3900
@@
 F 0 "R203" H 7230 3920 50  0000 L CNN
 F 1 "50R" H 7230 3860 50  0000 L CNN
-F 2 "" H 7200 3900 50  0000 C CNN
+F 2 "Resistors_SMD:R_0805_HandSoldering" H 7200 3900 50  0001 C CNN
 F 3 "" H 7200 3900 50  0000 C CNN
 	1    7200 3900
@@
 	7200 3350 7950 3350
 $Comp
-L GND #PWR204
+L GND #PWR012
 U 1 1 57EDA76C
 P 4650 3350
-F 0 "#PWR204" H 4650 3100 50  0001 C CNN
+F 0 "#PWR012" H 4650 3100 50  0001 C CNN
 F 1 "GND" H 4650 3200 50  0000 C CNN
 F 2 "" H 4650 3350 50  0000 C CNN

Commit message: Changed SWR microstrip for two transformers and gave missing values for components
Parts:
- C201, C202: value 1µF -> 100nF
- C203: value C_Small -> 1nF
Changed lines of the file:
@@
 U 1 1 57E31A00
 P 7600 3900
-F 0 "R205" H 7630 3920 50  0000 L CNN
-F 1 "50R" H 7630 3860 50  0000 L CNN
+F 0 "R205" V 7700 3900 50  0000 L CNN
+F 1 "50R" H 7600 3800 50  0000 L CNN
 F 2 "Resistors_SMD:R_0805_HandSoldering" H 7600 3900 50  0001 C CNN
 F 3 "" H 7600 3900 50  0000 C CNN
@@
 1,8Vrail
 $Comp
-L +Vlogic #PWR05
+L +Vlogic #PWR202
 U 1 1 57E31A13
 P 4350 2850
-F 0 "#PWR05" H 4350 2650 50  0001 C CNN
+F 0 "#PWR202" H 4350 2650 50  0001 C CNN
 F 1 "+Vlogic" H 4350 3050 50  0000 C CNN
 F 2 "" H 4350 2850 50  0000 C CNN
@@
 P 5100 3550
 F 0 "C202" H 5110 3620 50  0000 L CNN
-F 1 "1µF" H 5110 3470 50  0000 L CNN
+F 1 "100nF" H 5110 3470 50  0000 L CNN
 F 2 "Capacitors_SMD:C_0805" H 5100 3550 50  0001 C CNN
 F 3 "" H 5100 3550 50  0000 C CNN
@@
 P 4350 3150
 F 0 "C201" H 4360 3220 50  0000 L CNN
-F 1 "1µF" H 4360 3070 50  0000 L CNN
+F 1 "100nF" H 4360 3070 50  0000 L CNN
 F 2 "Capacitors_SMD:C_0805" H 4350 3150 50  0001 C CNN
 F 3 "" H 4350 3150 50  0000 C CNN
@@
 $EndComp
 $Comp
-L GND #PWR06
+L GND #PWR203
 U 1 1 57E31A2E
 P 4350 4200
-F 0 "#PWR06" H 4350 3950 50  0001 C CNN
+F 0 "#PWR203" H 4350 3950 50  0001 C CNN
 F 1 "GND" H 4350 4050 50  0000 C CNN
 F 2 "" H 4350 4200 50  0000 C CNN
@@
 $EndComp
 $Comp
-L +Vlogic #PWR07
+L +Vlogic #PWR201
 U 1 1 57E31A3B
 P 3750 3950
-F 0 "#PWR07" H 3750 3750 50  0001 C CNN
+F 0 "#PWR201" H 3750 3750 50  0001 C CNN
 F 1 "+Vlogic" H 3750 4150 50  0000 C CNN
 F 2 "" H 3750 3950 50  0000 C CNN
@@
 $EndComp
 $Comp
-L +Vlogic #PWR08
+L +Vlogic #PWR207
 U 1 1 57E31A41
 P 8050 3950
-F 0 "#PWR08" H 8050 3750 50  0001 C CNN
+F 0 "#PWR207" H 8050 3750 50  0001 C CNN
 F 1 "+Vlogic" H 8050 4150 50  0000 C CNN
 F 2 "" H 8050 3950 50  0000 C CNN
@@
 P 5700 4200
 F 0 "C203" H 5710 4270 50  0000 L CNN
-F 1 "C_Small" H 5710 4120 50  0000 L CNN
+F 1 "1nF" H 5710 4120 50  0000 L CNN
 F 2 "Capacitors_SMD:C_0805" H 5700 4200 50  0001 C CNN
 F 3 "" H 5700 4200 50  0000 C CNN
@@
 $EndComp
 $Comp
-L +Vlogic #PWR09
+L +Vlogic #PWR206
 U 1 1 57E31A5D
 P 6050 3550
-F 0 "#PWR09" H 6050 3350 50  0001 C CNN
+F 0 "#PWR206" H 6050 3350 50  0001 C CNN
 F 1 "+Vlogic" H 6050 3750 50  0000 C CNN
 F 2 "" H 6050 3550 50  0000 C CNN
@@
 $EndComp
 $Comp
-L GND #PWR010
+L GND #PWR205
 U 1 1 57E31A71
 P 5900 3950
-F 0 "#PWR010" H 5900 3700 50  0001 C CNN
+F 0 "#PWR205" H 5900 3700 50  0001 C CNN
 F 1 "GND" H 5900 3800 50  0000 C CNN
 F 2 "" H 5900 3950 50  0000 C CNN
@@
 $EndComp
 $Comp
-L GND #PWR011
+L GND #PWR208
 U 1 1 57E31A77
 P 8050 4200
-F 0 "#PWR011" H 8050 3950 50  0001 C CNN
+F 0 "#PWR208" H 8050 3950 50  0001 C CNN
 F 1 "GND" H 8050 4050 50  0000 C CNN
 F 2 "" H 8050 4200 50  0000 C CNN
@@
 U 1 1 57E545D0
 P 7400 3900
-F 0 "R204" H 7430 3920 50  0000 L CNN
-F 1 "50R" H 7430 3860 50  0000 L CNN
+F 0 "R204" V 7500 3900 50  0000 L CNN
+F 1 "50R" H 7400 3800 50  0000 L CNN
 F 2 "Resistors_SMD:R_0805_HandSoldering" H 7400 3900 50  0001 C CNN
 F 3 "" H 7400 3900 50  0000 C CNN
@@
 U 1 1 57E54652
 P 7200 3900
-F 0 "R203" H 7230 3920 50  0000 L CNN
-F 1 "50R" H 7230 3860 50  0000 L CNN
+F 0 "R203" V 7300 3900 50  0000 L CNN
+F 1 "50R" H 7200 3800 50  0000 L CNN
 F 2 "Resistors_SMD:R_0805_HandSoldering" H 7200 3900 50  0001 C CNN
 F 3 "" H 7200 3900 50  0000 C CNN
@@
 	7200 3350 7950 3350
 $Comp
-L GND #PWR012
+L GND #PWR204
 U 1 1 57EDA76C
 P 4650 3350
-F 0 "#PWR012" H 4650 3100 50  0001 C CNN
+F 0 "#PWR204" H 4650 3100 50  0001 C CNN
 F 1 "GND" H 4650 3200 50  0000 C CNN
 F 2 "" H 4650 3350 50  0000 C CNN

Commit message: Fixed some bugs and annotated rest of the footprints
Parts:
- C201, C202, C203, C204, C205: footprint Capacitors_SMD:C_0805 -> Capacitors_SMD:C_0805_HandSoldering
- OSC201: footprint (none) -> dodekaedri:TCXO_1.5x2mm
- U201: footprint (none) -> TO_SOT_Packages_SMD:SOT-23-5
- U202: footprint (none) -> Housings_SSOP:MSOP-10_3x3mm_Pitch0.5mm
Changed lines of the file:
@@
 1,8Vrail
 $Comp
-L +Vlogic #PWR202
+L +Vlogic #PWR04
 U 1 1 57E31A13
 P 4350 2850
-F 0 "#PWR202" H 4350 2650 50  0001 C CNN
+F 0 "#PWR04" H 4350 2650 50  0001 C CNN
 F 1 "+Vlogic" H 4350 3050 50  0000 C CNN
 F 2 "" H 4350 2850 50  0000 C CNN
@@
 F 0 "C202" H 5110 3620 50  0000 L CNN
 F 1 "100nF" H 5110 3470 50  0000 L CNN
-F 2 "Capacitors_SMD:C_0805" H 5100 3550 50  0001 C CNN
+F 2 "Capacitors_SMD:C_0805_HandSoldering" H 5100 3550 50  0001 C CNN
 F 3 "" H 5100 3550 50  0000 C CNN
 	1    5100 3550
@@
 F 0 "C201" H 4360 3220 50  0000 L CNN
 F 1 "100nF" H 4360 3070 50  0000 L CNN
-F 2 "Capacitors_SMD:C_0805" H 4350 3150 50  0001 C CNN
+F 2 "Capacitors_SMD:C_0805_HandSoldering" H 4350 3150 50  0001 C CNN
 F 3 "" H 4350 3150 50  0000 C CNN
 	1    4350 3150
@@
 F 0 "U201" H 5100 2800 60  0000 C CNN
 F 1 "MIC5365" H 5100 3300 60  0000 C CNN
-F 2 "" H 5100 3050 60  0001 C CNN
+F 2 "TO_SOT_Packages_SMD:SOT-23-5" H 5100 3050 60  0001 C CNN
 F 3 "" H 5100 3050 60  0001 C CNN
 	1    5100 3100
@@
 $EndComp
 $Comp
-L GND #PWR203
+L GND #PWR05
 U 1 1 57E31A2E
 P 4350 4200
-F 0 "#PWR203" H 4350 3950 50  0001 C CNN
+F 0 "#PWR05" H 4350 3950 50  0001 C CNN
 F 1 "GND" H 4350 4050 50  0000 C CNN
 F 2 "" H 4350 4200 50  0000 C CNN
@@
 F 0 "OSC201" H 5000 3800 60  0000 C CNN
 F 1 "TCXO 26MHz" H 5000 4300 60  0000 C CNN
-F 2 "" H 5050 4150 60  0001 C CNN
+F 2 "dodekaedri:TCXO_1.5x2mm" H 5050 4150 60  0001 C CNN
 F 3 "" H 5050 4150 60  0001 C CNN
 	1    5000 4050
@@
 $EndComp
 $Comp
-L +Vlogic #PWR201
+L +Vlogic #PWR06
 U 1 1 57E31A3B
 P 3750 3950
-F 0 "#PWR201" H 3750 3750 50  0001 C CNN
+F 0 "#PWR06" H 3750 3750 50  0001 C CNN
 F 1 "+Vlogic" H 3750 4150 50  0000 C CNN
 F 2 "" H 3750 3950 50  0000 C CNN
@@
 $EndComp
 $Comp
-L +Vlogic #PWR207
+L +Vlogic #PWR07
 U 1 1 57E31A41
 P 8050 3950
-F 0 "#PWR207" H 8050 3750 50  0001 C CNN
+F 0 "#PWR07" H 8050 3750 50  0001 C CNN
 F 1 "+Vlogic" H 8050 4150 50  0000 C CNN
 F 2 "" H 8050 3950 50  0000 C CNN
@@
 F 0 "C203" H 5710 4270 50  0000 L CNN
 F 1 "1nF" H 5710 4120 50  0000 L CNN
-F 2 "Capacitors_SMD:C_0805" H 5700 4200 50  0001 C CNN
+F 2 "Capacitors_SMD:C_0805_HandSoldering" H 5700 4200 50  0001 C CNN
 F 3 "" H 5700 4200 50  0000 C CNN
 	1    5700 4200
@@
 $EndComp
 $Comp
-L +Vlogic #PWR206
+L +Vlogic #PWR08
 U 1 1 57E31A5D
 P 6050 3550
-F 0 "#PWR206" H 6050 3350 50  0001 C CNN
+F 0 "#PWR08" H 6050 3350 50  0001 C CNN
 F 1 "+Vlogic" H 6050 3750 50  0000 C CNN
 F 2 "" H 6050 3550 50  0000 C CNN
@@
 F 0 "C205" H 8060 4170 50  0000 L CNN
 F 1 "100nF" H 8060 4020 50  0000 L CNN
-F 2 "Capacitors_SMD:C_0805" H 8050 4100 50  0001 C CNN
+F 2 "Capacitors_SMD:C_0805_HandSoldering" H 8050 4100 50  0001 C CNN
 F 3 "" H 8050 4100 50  0000 C CNN
 	1    8050 4100
@@
 F 0 "C204" H 5910 3870 50  0000 L CNN
 F 1 "100nF" H 5910 3720 50  0000 L CNN
-F 2 "Capacitors_SMD:C_0805" H 5900 3800 50  0001 C CNN
+F 2 "Capacitors_SMD:C_0805_HandSoldering" H 5900 3800 50  0001 C CNN
 F 3 "" H 5900 3800 50  0000 C CNN
 	1    5900 3800
@@
 $EndComp
 $Comp
-L GND #PWR205
+L GND #PWR09
 U 1 1 57E31A71
 P 5900 3950
-F 0 "#PWR205" H 5900 3700 50  0001 C CNN
+F 0 "#PWR09" H 5900 3700 50  0001 C CNN
 F 1 "GND" H 5900 3800 50  0000 C CNN
 F 2 "" H 5900 3950 50  0000 C CNN
@@
 $EndComp
 $Comp
-L GND #PWR208
+L GND #PWR010
 U 1 1 57E31A77
 P 8050 4200
-F 0 "#PWR208" H 8050 3950 50  0001 C CNN
+F 0 "#PWR010" H 8050 3950 50  0001 C CNN
 F 1 "GND" H 8050 4050 50  0000 C CNN
 F 2 "" H 8050 4200 50  0000 C CNN
@@
 F 0 "U202" H 6650 3950 60  0000 C CNN
 F 1 "SI5351A" H 6650 4650 60  0000 C CNN
-F 2 "" H 6650 4650 60  0001 C CNN
+F 2 "Housings_SSOP:MSOP-10_3x3mm_Pitch0.5mm" H 6650 4650 60  0001 C CNN
 F 3 "" H 6650 4650 60  0001 C CNN
 	1    6650 4300
@@
 	7200 3350 7950 3350
 $Comp
-L GND #PWR204
+L GND #PWR011
 U 1 1 57EDA76C
 P 4650 3350
-F 0 "#PWR204" H 4650 3100 50  0001 C CNN
+F 0 "#PWR011" H 4650 3100 50  0001 C CNN
 F 1 "GND" H 4650 3200 50  0000 C CNN
 F 2 "" H 4650 3350 50  0000 C CNN

Commit message: Changed some component values
Parts:
- R201, R202: value 10k -> 1k
- R203, R204, R205, R206, R207: value 50R -> 100R
Changed lines of the file:
@@
 P 7800 4500
 F 0 "R207" H 7830 4520 50  0000 L CNN
-F 1 "50R" H 7830 4460 50  0000 L CNN
+F 1 "100R" H 7830 4460 50  0000 L CNN
 F 2 "Resistors_SMD:R_0805_HandSoldering" H 7800 4500 50  0001 C CNN
 F 3 "" H 7800 4500 50  0000 C CNN
@@
 P 7600 3900
 F 0 "R205" V 7700 3900 50  0000 L CNN
-F 1 "50R" H 7600 3800 50  0000 L CNN
+F 1 "100R" H 7600 3800 50  0000 L CNN
 F 2 "Resistors_SMD:R_0805_HandSoldering" H 7600 3900 50  0001 C CNN
 F 3 "" H 7600 3900 50  0000 C CNN
@@
 P 7800 3900
 F 0 "R206" H 7830 3920 50  0000 L CNN
-F 1 "50R" H 7830 3860 50  0000 L CNN
+F 1 "100R" H 7830 3860 50  0000 L CNN
 F 2 "Resistors_SMD:R_0805_HandSoldering" H 7800 3900 50  0001 C CNN
 F 3 "" H 7800 3900 50  0000 C CNN
@@
 P 3600 4100
 F 0 "R201" V 3680 4100 50  0000 C CNN
-F 1 "10k" V 3600 4100 50  0000 C CNN
+F 1 "1k" V 3600 4100 50  0000 C CNN
 F 2 "Resistors_SMD:R_0805_HandSoldering" V 3530 4100 50  0001 C CNN
 F 3 "" H 3600 4100 50  0000 C CNN
@@
 P 3900 4100
 F 0 "R202" V 3980 4100 50  0000 C CNN
-F 1 "10k" V 3900 4100 50  0000 C CNN
+F 1 "1k" V 3900 4100 50  0000 C CNN
 F 2 "Resistors_SMD:R_0805_HandSoldering" V 3830 4100 50  0001 C CNN
 F 3 "" H 3900 4100 50  0000 C CNN
@@
 P 7400 3900
 F 0 "R204" V 7500 3900 50  0000 L CNN
-F 1 "50R" H 7400 3800 50  0000 L CNN
+F 1 "100R" H 7400 3800 50  0000 L CNN
 F 2 "Resistors_SMD:R_0805_HandSoldering" H 7400 3900 50  0001 C CNN
 F 3 "" H 7400 3900 50  0000 C CNN
@@
 P 7200 3900
 F 0 "R203" V 7300 3900 50  0000 L CNN
-F 1 "50R" H 7200 3800 50  0000 L CNN
+F 1 "100R" H 7200 3800 50  0000 L CNN
 F 2 "Resistors_SMD:R_0805_HandSoldering" H 7200 3900 50  0001 C CNN
 F 3 "" H 7200 3900 50  0000 C CNN
