File: hardware/cpu.sch (KiCad schematic (older format))
At the start: 105 parts, among them J801 HANDSFREE, J802 microphone, J803 HEADPHONES, P801 TX_SW_WIRE, P802 USB_OTG, P803 UART, P804 PROG, P805 RNG_PINS, P806 CONN_01X08, P807 CONN_01X04, P808 CONN_02X04, P809 BOOT0JMPR, Q801 BSS84, SW801 SW_PUSH, SW802 SW, SW803 SW, SW804 SW, SW805 SW, SW806 encoder, SW807 RESET, SW808 SW, SW809 encoder, SW810 SW, U801 STM32F401, U802 WM8731

Commit message: halfway through layout
Parts:
- removed D808, D811, D813, D815, D816, D817: 1N914, symbol D
- removed R817, R829: 50R, Resistors_SMD:R_0805_HandSoldering, symbol R
- removed SW805: SW, Buttons_Switches_SMD:SW_SPST_B3SL-1002P, symbol SW_PUSH_SMALL
- removed SW808, SW810: SW, symbol SW_PUSH_SMALL
- removed SW809: encoder, symbol encoder
- added R822: 10k, Resistors_SMD:R_0805_HandSoldering, symbol R
- D805, D806, D807, D809, D810, D812: footprint TO_SOT_Packages_SMD:SOT-23_Handsoldering -> dodekaedri:SOT-23_HS_2-1-3
- R808: value 47k -> 100k
- R813: value 1k -> 100k; footprint (none) -> Resistors_SMD:R_0805_HandSoldering
- R815: value 680R -> 1k
Connections:
- net PC3 is gone; now on net VIN_ADC: D823.3 (common), U801.11 (PC3)
- net GND: now also P805.3 (P3), R822.2
- net Vin_net: now also R813.1
- net at P808.6 (P6), U801.41 (PA8): no longer R813.1
- net VIN_ADC: now reaches R813.2
- net VIN_ADC: now also R822.1
Other:
- note added: "This is for the reference where 4th row of buttons\nand second encoder were ment to be connected"
- note removed: "connector block"
- moved on the sheet: D823

Commit message: All components are placed. GND and +Vlogic copper fills still undone
Parts:
- P802: symbol USB_OTG -> USB_OTG-RESCUE-dodekaedri
Changed lines of the file:
@@
 $EndComp
 $Comp
-L USB_OTG P802
+L USB_OTG-RESCUE-dodekaedri P802
 U 1 1 57F10790
 P 1400 7200

Commit message: Changed some component values
Parts:
- C804: value 1n -> 1nF
- D805, D806, D807, D809, D810, D812: value 1N914 -> BAT54SL
- D818, D819, D820, D821, D822, D823: value BAT54 -> BAT54SL
- R801, R805, R807: value 10k -> 100k
- R802, R804: value 100R -> 1k
- R810, R811: value 10k -> 0.1pF
- R812, R814, R816: value 10k -> 1k
- R818, R819, R823, R824: value 50R -> 100R
- R822: value 10k -> 7k87
Changed lines of the file:
@@
 P 6450 3100
 F 0 "R810" V 6530 3100 50  0000 C CNN
-F 1 "10k" V 6450 3100 50  0000 C CNN
+F 1 "0.1pF" V 6450 3100 50  0000 C CNN
 F 2 "Resistors_SMD:R_0805_HandSoldering" V 6380 3100 50  0001 C CNN
 F 3 "" H 6450 3100 50  0000 C CNN
@@
 P 6650 3100
 F 0 "R811" V 6730 3100 50  0000 C CNN
-F 1 "10k" V 6650 3100 50  0000 C CNN
+F 1 "0.1pF" V 6650 3100 50  0000 C CNN
 F 2 "Resistors_SMD:R_0805_HandSoldering" V 6580 3100 50  0001 C CNN
 F 3 "" H 6650 3100 50  0000 C CNN
@@
 P 6900 3050
 F 0 "R812" V 6980 3050 50  0000 C CNN
-F 1 "10k" V 6900 3050 50  0000 C CNN
+F 1 "1k" V 6900 3050 50  0000 C CNN
 F 2 "Resistors_SMD:R_0805_HandSoldering" V 6830 3050 50  0001 C CNN
 F 3 "" H 6900 3050 50  0000 C CNN
@@
 P 7400 3650
 F 0 "R816" V 7480 3650 50  0000 C CNN
-F 1 "10k" V 7400 3650 50  0000 C CNN
+F 1 "1k" V 7400 3650 50  0000 C CNN
 F 2 "Resistors_SMD:R_0805_HandSoldering" V 7330 3650 50  0001 C CNN
 F 3 "" H 7400 3650 50  0000 C CNN
@@
 P 7850 4450
 F 0 "R818" V 7930 4450 50  0000 C CNN
-F 1 "50R" V 7850 4450 50  0000 C CNN
+F 1 "100R" V 7850 4450 50  0000 C CNN
 F 2 "Resistors_SMD:R_0805_HandSoldering" V 7780 4450 50  0001 C CNN
 F 3 "" H 7850 4450 50  0000 C CNN
@@
 P 7000 1900
 F 0 "R814" V 7080 1900 50  0000 C CNN
-F 1 "10k" V 7000 1900 50  0000 C CNN
+F 1 "1k" V 7000 1900 50  0000 C CNN
 F 2 "Resistors_SMD:R_0805_HandSoldering" V 6930 1900 50  0001 C CNN
 F 3 "" H 7000 1900 50  0000 C CNN
@@
 P 1100 3550
 F 0 "R801" V 1180 3550 50  0000 C CNN
-F 1 "10k" V 1100 3550 50  0000 C CNN
+F 1 "100k" V 1100 3550 50  0000 C CNN
 F 2 "Resistors_SMD:R_0805_HandSoldering" V 1030 3550 50  0001 C CNN
 F 3 "" H 1100 3550 50  0000 C CNN
@@
 P 1850 3850
 F 0 "C804" V 1900 3900 50  0000 L CNN
-F 1 "1n" H 1875 3750 50  0000 L CNN
+F 1 "1nF" H 1875 3750 50  0000 L CNN
 F 2 "Capacitors_SMD:C_0805_HandSoldering" H 1888 3700 50  0001 C CNN
 F 3 "" H 1850 3850 50  0000 C CNN
@@
 P 1650 3550
 F 0 "R802" V 1730 3550 50  0000 C CNN
-F 1 "100R" V 1650 3550 50  0000 C CNN
+F 1 "1k" V 1650 3550 50  0000 C CNN
 F 2 "Resistors_SMD:R_0805_HandSoldering" V 1580 3550 50  0001 C CNN
 F 3 "" H 1650 3550 50  0000 C CNN
@@
 P 2000 4650
 F 0 "R804" V 2080 4650 50  0000 C CNN
-F 1 "100R" V 2000 4650 50  0000 C CNN
+F 1 "1k" V 2000 4650 50  0000 C CNN
 F 2 "Resistors_SMD:R_0805_HandSoldering" V 1930 4650 50  0001 C CNN
 F 3 "" H 2000 4650 50  0000 C CNN
@@
 P 4950 6150
 F 0 "D805" H 4950 6250 50  0000 C CNN
-F 1 "1N914" H 4950 6050 50  0000 C CNN
+F 1 "BAT54SL" H 4950 6050 50  0000 C CNN
 F 2 "dodekaedri:SOT-23_HS_2-1-3" H 4950 6150 50  0001 C CNN
 F 3 "" H 4950 6150 50  0000 C CNN
@@
 P 4950 6650
 F 0 "D806" H 4950 6750 50  0000 C CNN
-F 1 "1N914" H 5000 6550 50  0000 C CNN
+F 1 "BAT54SL" H 5000 6550 50  0000 C CNN
 F 2 "dodekaedri:SOT-23_HS_2-1-3" H 4950 6650 50  0001 C CNN
 F 3 "" H 4950 6650 50  0000 C CNN
@@
 P 4950 7100
 F 0 "D807" H 4950 7200 50  0000 C CNN
-F 1 "1N914" H 4950 7000 50  0000 C CNN
+F 1 "BAT54SL" H 4950 7000 50  0000 C CNN
 F 2 "dodekaedri:SOT-23_HS_2-1-3" H 4950 7100 50  0001 C CNN
 F 3 "" H 4950 7100 50  0000 C CNN
@@
 P 5500 6100
 F 0 "D809" H 5500 6200 50  0000 C CNN
-F 1 "1N914" H 5500 6000 50  0000 C CNN
+F 1 "BAT54SL" H 5500 6000 50  0000 C CNN
 F 2 "dodekaedri:SOT-23_HS_2-1-3" H 5500 6100 50  0001 C CNN
 F 3 "" H 5500 6100 50  0000 C CNN
@@
 P 5950 7050
 F 0 "D812" H 5950 7150 50  0000 C CNN
-F 1 "1N914" H 5950 6950 50  0000 C CNN
+F 1 "BAT54SL" H 5950 6950 50  0000 C CNN
 F 2 "dodekaedri:SOT-23_HS_2-1-3" H 5950 7050 50  0001 C CNN
 F 3 "" H 5950 7050 50  0000 C CNN
@@
 P 5750 6600
 F 0 "D810" H 5750 6700 50  0000 C CNN
-F 1 "1N914" H 5750 6500 50  0000 C CNN
+F 1 "BAT54SL" H 5750 6500 50  0000 C CNN
 F 2 "dodekaedri:SOT-23_HS_2-1-3" H 5750 6600 50  0001 C CNN
 F 3 "" H 5750 6600 50  0000 C CNN
@@
 P 8200 4050
 F 0 "R819" V 8280 4050 50  0000 C CNN
-F 1 "50R" V 8200 4050 50  0000 C CNN
+F 1 "100R" V 8200 4050 50  0000 C CNN
 F 2 "Resistors_SMD:R_0805_HandSoldering" V 8130 4050 50  0001 C CNN
 F 3 "" H 8200 4050 50  0000 C CNN
@@
 P 4900 850
 F 0 "R805" V 4980 850 50  0000 C CNN
-F 1 "10k" V 4900 850 50  0000 C CNN
+F 1 "100k" V 4900 850 50  0000 C CNN
 F 2 "Resistors_SMD:R_0805_HandSoldering" V 4830 850 50  0001 C CNN
 F 3 "" H 4900 850 50  0000 C CNN
@@
 P 5800 750
 F 0 "R807" V 5880 750 50  0000 C CNN
-F 1 "10k" V 5800 750 50  0000 C CNN
+F 1 "100k" V 5800 750 50  0000 C CNN
 F 2 "Resistors_SMD:R_0805_HandSoldering" V 5730 750 50  0001 C CNN
 F 3 "" H 5800 750 50  0000 C CNN
@@
 P 7600 5750
 F 0 "D823" H 7700 5650 50  0000 C CNN
-F 1 "BAT54" H 7600 5850 50  0000 C CNN
+F 1 "BAT54SL" H 7600 5850 50  0000 C CNN
 F 2 "TO_SOT_Packages_SMD:SOT-23_Handsoldering" H 7600 5750 50  0001 C CNN
 F 3 "" H 7600 5750 50  0000 C CNN
@@
 P 1800 5600
 F 0 "D819" H 1900 5500 50  0000 C CNN
-F 1 "BAT54" H 1800 5700 50  0000 C CNN
+F 1 "BAT54SL" H 1800 5700 50  0000 C CNN
 F 2 "TO_SOT_Packages_SMD:SOT-23_Handsoldering" H 1800 5600 50  0001 C CNN
 F 3 "" H 1800 5600 50  0000 C CNN
@@
 P 2200 6000
 F 0 "D820" H 2300 5900 50  0000 C CNN
-F 1 "BAT54" H 2200 6100 50  0000 C CNN
+F 1 "BAT54SL" H 2200 6100 50  0000 C CNN
 F 2 "TO_SOT_Packages_SMD:SOT-23_Handsoldering" H 2200 6000 50  0001 C CNN
 F 3 "" H 2200 6000 50  0000 C CNN
@@
 P 3200 5600
 F 0 "D822" H 3300 5500 50  0000 C CNN
-F 1 "BAT54" H 3200 5700 50  0000 C CNN
+F 1 "BAT54SL" H 3200 5700 50  0000 C CNN
 F 2 "TO_SOT_Packages_SMD:SOT-23_Handsoldering" H 3200 5600 50  0001 C CNN
 F 3 "" H 3200 5600 50  0000 C CNN
@@
 P 2800 6200
 F 0 "D821" H 2700 6100 50  0000 C CNN
-F 1 "BAT54" H 2800 6300 50  0000 C CNN
+F 1 "BAT54SL" H 2800 6300 50  0000 C CNN
 F 2 "TO_SOT_Packages_SMD:SOT-23_Handsoldering" H 2800 6200 50  0001 C CNN
 F 3 "" H 2800 6200 50  0000 C CNN
@@
 P 1300 6200
 F 0 "R823" V 1250 6400 50  0000 C CNN
-F 1 "50R" V 1300 6200 50  0000 C CNN
+F 1 "100R" V 1300 6200 50  0000 C CNN
 F 2 "Resistors_SMD:R_0805_HandSoldering" V 1230 6200 50  0001 C CNN
 F 3 "" H 1300 6200 50  0000 C CNN
@@
 P 1300 6300
 F 0 "R824" V 1250 6500 50  0000 C CNN
-F 1 "50R" V 1300 6300 50  0000 C CNN
+F 1 "100R" V 1300 6300 50  0000 C CNN
 F 2 "Resistors_SMD:R_0805_HandSoldering" V 1230 6300 50  0001 C CNN
 F 3 "" H 1300 6300 50  0000 C CNN
@@
 P 650 3900
 F 0 "D818" H 700 3800 50  0000 C CNN
-F 1 "BAT54" H 650 4000 50  0000 C CNN
+F 1 "BAT54SL" H 650 4000 50  0000 C CNN
 F 2 "TO_SOT_Packages_SMD:SOT-23_Handsoldering" H 650 3900 50  0001 C CNN
 F 3 "" H 650 3900 50  0000 C CNN
@@
 P 7300 5900
 F 0 "R822" V 7380 5900 50  0000 C CNN
-F 1 "10k" V 7300 5900 50  0000 C CNN
+F 1 "7k87" V 7300 5900 50  0000 C CNN
 F 2 "Resistors_SMD:R_0805_HandSoldering" V 7230 5900 50  0001 C CNN
 F 3 "" H 7300 5900 50  0000 C CNN
