File: hardware/radio_conv.sch (KiCad schematic (older format))
At the start: 10 parts, among them U701 WM8731, U702 MCP6L02

Commit message: Linked first components to footprints and updated schematic plot
Parts:
- C701, C702, C703, C704, C705: footprint (none) -> Capacitors_SMD:C_0805
- R701, R702, R703: footprint (none) -> Resistors_SMD:R_0805_HandSoldering
- U701: footprint (none) -> Housings_SSOP:SSOP-28_5.3x10.2mm_Pitch0.65mm
- U702: footprint (none) -> Housings_SOIC:SOIC-8_3.9x4.9mm_Pitch1.27mm
Changed lines of the file:
@@
 F 0 "U701" H 5800 3450 60  0000 C CNN
 F 1 "WM8731" H 5800 3800 60  0000 C CNN
-F 2 "" H 5800 4050 60  0001 C CNN
+F 2 "Housings_SSOP:SSOP-28_5.3x10.2mm_Pitch0.65mm" H 5800 4050 60  0001 C CNN
 F 3 "" H 5800 4050 60  0001 C CNN
 	1    5800 3600
@@
 $EndComp
 $Comp
-L +Vlogic #PWR704
+L +Vlogic #PWR046
 U 1 1 57E4C112
 P 5800 2200
-F 0 "#PWR704" H 5800 2000 50  0001 C CNN
+F 0 "#PWR046" H 5800 2000 50  0001 C CNN
 F 1 "+Vlogic" H 5800 2400 50  0000 C CNN
 F 2 "" H 5800 2200 50  0000 C CNN
@@
 F 0 "C701" H 4700 2550 50  0000 L CNN
 F 1 "10µF" H 4700 2350 50  0000 L CNN
-F 2 "" H 4713 2300 50  0000 C CNN
+F 2 "Capacitors_SMD:C_0805" H 4713 2300 50  0001 C CNN
 F 3 "" H 4675 2450 50  0000 C CNN
 	1    4675 2450
@@
 F 0 "C702" H 4700 2850 50  0000 L CNN
 F 1 "10µF" H 4700 2650 50  0000 L CNN
-F 2 "" H 4713 2600 50  0000 C CNN
+F 2 "Capacitors_SMD:C_0805" H 4713 2600 50  0001 C CNN
 F 3 "" H 4675 2750 50  0000 C CNN
 	1    4675 2750
@@
 $EndComp
 $Comp
-L GND #PWR701
+L GND #PWR047
 U 1 1 57E4C149
 P 4300 2600
-F 0 "#PWR701" H 4300 2350 50  0001 C CNN
+F 0 "#PWR047" H 4300 2350 50  0001 C CNN
 F 1 "GND" H 4300 2450 50  0000 C CNN
 F 2 "" H 4300 2600 50  0000 C CNN
@@
 F 0 "C703" H 6725 2600 50  0000 L CNN
 F 1 "10µF" H 6725 2400 50  0000 L CNN
-F 2 "" H 6738 2350 50  0000 C CNN
+F 2 "Capacitors_SMD:C_0805" H 6738 2350 50  0001 C CNN
 F 3 "" H 6700 2500 50  0000 C CNN
 	1    6700 2500
@@
 F 0 "C704" H 6725 3050 50  0000 L CNN
 F 1 "10µF" H 6725 2850 50  0000 L CNN
-F 2 "" H 6738 2800 50  0000 C CNN
+F 2 "Capacitors_SMD:C_0805" H 6738 2800 50  0001 C CNN
 F 3 "" H 6700 2950 50  0000 C CNN
 	1    6700 2950
@@
 Connection ~ 6700 2650
 $Comp
-L GND #PWR706
+L GND #PWR048
 U 1 1 57E4C178
 P 7225 2650
-F 0 "#PWR706" H 7225 2400 50  0001 C CNN
+F 0 "#PWR048" H 7225 2400 50  0001 C CNN
 F 1 "GND" H 7225 2500 50  0000 C CNN
 F 2 "" H 7225 2650 50  0000 C CNN
@@
 Connection ~ 4675 2200
 $Comp
-L +Vlogic #PWR702
+L +Vlogic #PWR049
 U 1 1 57E4C199
 P 4550 4300
-F 0 "#PWR702" H 4550 4100 50  0001 C CNN
+F 0 "#PWR049" H 4550 4100 50  0001 C CNN
 F 1 "+Vlogic" H 4550 4450 50  0000 C CNN
 F 2 "" H 4550 4300 50  0000 C CNN
@@
 F 0 "R701" V 4530 4450 50  0000 C CNN
 F 1 "10k" V 4450 4450 50  0000 C CNN
-F 2 "" V 4380 4450 50  0000 C CNN
+F 2 "Resistors_SMD:R_0805_HandSoldering" V 4380 4450 50  0001 C CNN
 F 3 "" H 4450 4450 50  0000 C CNN
 	1    4450 4450
@@
 F 0 "R702" V 4730 4450 50  0000 C CNN
 F 1 "10k" V 4650 4450 50  0000 C CNN
-F 2 "" V 4580 4450 50  0000 C CNN
+F 2 "Resistors_SMD:R_0805_HandSoldering" V 4580 4450 50  0001 C CNN
 F 3 "" H 4650 4450 50  0000 C CNN
 	1    4650 4450
@@
 F 0 "C705" H 6875 4700 50  0000 L CNN
 F 1 "10µF" H 6875 4500 50  0000 L CNN
-F 2 "" H 6888 4450 50  0000 C CNN
+F 2 "Capacitors_SMD:C_0805" H 6888 4450 50  0001 C CNN
 F 3 "" H 6850 4600 50  0000 C CNN
 	1    6850 4600
@@
 	6850 4750 7550 4750
 $Comp
-L GND #PWR705
+L GND #PWR050
 U 1 1 57E4C1C1
 P 7100 4750
-F 0 "#PWR705" H 7100 4500 50  0001 C CNN
+F 0 "#PWR050" H 7100 4500 50  0001 C CNN
 F 1 "GND" H 7100 4600 50  0000 C CNN
 F 2 "" H 7100 4750 50  0000 C CNN
@@
 RX_Q
 $Comp
-L GND #PWR703
+L GND #PWR051
 U 1 1 57E4C1DF
 P 5000 5200
-F 0 "#PWR703" H 5000 4950 50  0001 C CNN
+F 0 "#PWR051" H 5000 4950 50  0001 C CNN
 F 1 "GND" H 5000 5050 50  0000 C CNN
 F 2 "" H 5000 5200 50  0000 C CNN
@@
 F 0 "U702" H 8050 4300 60  0000 C CNN
 F 1 "MCP6L02" H 8050 4900 60  0000 C CNN
-F 2 "" H 8100 4600 60  0001 C CNN
+F 2 "Housings_SOIC:SOIC-8_3.9x4.9mm_Pitch1.27mm" H 8100 4600 60  0001 C CNN
 F 3 "" H 8100 4600 60  0001 C CNN
 	1    8050 4600
@@
 	8550 4550 8550 4650
 $Comp
-L +Vlogic #PWR707
+L +Vlogic #PWR052
 U 1 1 57E46B0D
 P 8550 4150
-F 0 "#PWR707" H 8550 3950 50  0001 C CNN
+F 0 "#PWR052" H 8550 3950 50  0001 C CNN
 F 1 "+Vlogic" H 8550 4350 50  0000 C CNN
 F 2 "" H 8550 4150 50  0000 C CNN
@@
 F 0 "R703" V 5080 5000 50  0000 C CNN
 F 1 "10k" V 5000 5000 50  0000 C CNN
-F 2 "" V 4930 5000 50  0000 C CNN
+F 2 "Resistors_SMD:R_0805_HandSoldering" V 4930 5000 50  0001 C CNN
 F 3 "" H 5000 5000 50  0000 C CNN
 	1    5000 5000

Commit message: Fixed some bugs and annotated rest of the footprints
Parts:
- C701, C702, C703, C704, C705: footprint Capacitors_SMD:C_0805 -> Capacitors_SMD:C_0805_HandSoldering
Changed lines of the file:
@@
 $EndComp
 $Comp
-L +Vlogic #PWR704
+L +Vlogic #PWR044
 U 1 1 57E4C112
 P 5800 2200
-F 0 "#PWR704" H 5800 2000 50  0001 C CNN
+F 0 "#PWR044" H 5800 2000 50  0001 C CNN
 F 1 "+Vlogic" H 5800 2400 50  0000 C CNN
 F 2 "" H 5800 2200 50  0000 C CNN
@@
 F 0 "C701" H 4700 2550 50  0000 L CNN
 F 1 "10µF" H 4700 2350 50  0000 L CNN
-F 2 "Capacitors_SMD:C_0805" H 4713 2300 50  0001 C CNN
+F 2 "Capacitors_SMD:C_0805_HandSoldering" H 4713 2300 50  0001 C CNN
 F 3 "" H 4675 2450 50  0000 C CNN
 	1    4675 2450
@@
 F 0 "C702" H 4700 2850 50  0000 L CNN
 F 1 "10µF" H 4700 2650 50  0000 L CNN
-F 2 "Capacitors_SMD:C_0805" H 4713 2600 50  0001 C CNN
+F 2 "Capacitors_SMD:C_0805_HandSoldering" H 4713 2600 50  0001 C CNN
 F 3 "" H 4675 2750 50  0000 C CNN
 	1    4675 2750
@@
 $EndComp
 $Comp
-L GND #PWR701
+L GND #PWR045
 U 1 1 57E4C149
 P 4300 2600
-F 0 "#PWR701" H 4300 2350 50  0001 C CNN
+F 0 "#PWR045" H 4300 2350 50  0001 C CNN
 F 1 "GND" H 4300 2450 50  0000 C CNN
 F 2 "" H 4300 2600 50  0000 C CNN
@@
 F 0 "C703" H 6725 2600 50  0000 L CNN
 F 1 "10µF" H 6725 2400 50  0000 L CNN
-F 2 "Capacitors_SMD:C_0805" H 6738 2350 50  0001 C CNN
+F 2 "Capacitors_SMD:C_0805_HandSoldering" H 6738 2350 50  0001 C CNN
 F 3 "" H 6700 2500 50  0000 C CNN
 	1    6700 2500
@@
 F 0 "C704" H 6725 3050 50  0000 L CNN
 F 1 "10µF" H 6725 2850 50  0000 L CNN
-F 2 "Capacitors_SMD:C_0805" H 6738 2800 50  0001 C CNN
+F 2 "Capacitors_SMD:C_0805_HandSoldering" H 6738 2800 50  0001 C CNN
 F 3 "" H 6700 2950 50  0000 C CNN
 	1    6700 2950
@@
 Connection ~ 6700 2650
 $Comp
-L GND #PWR706
+L GND #PWR046
 U 1 1 57E4C178
 P 7225 2650
-F 0 "#PWR706" H 7225 2400 50  0001 C CNN
+F 0 "#PWR046" H 7225 2400 50  0001 C CNN
 F 1 "GND" H 7225 2500 50  0000 C CNN
 F 2 "" H 7225 2650 50  0000 C CNN
@@
 Connection ~ 4675 2200
 $Comp
-L +Vlogic #PWR702
+L +Vlogic #PWR047
 U 1 1 57E4C199
 P 4550 4300
-F 0 "#PWR702" H 4550 4100 50  0001 C CNN
+F 0 "#PWR047" H 4550 4100 50  0001 C CNN
 F 1 "+Vlogic" H 4550 4450 50  0000 C CNN
 F 2 "" H 4550 4300 50  0000 C CNN
@@
 F 0 "C705" H 6875 4700 50  0000 L CNN
 F 1 "10µF" H 6875 4500 50  0000 L CNN
-F 2 "Capacitors_SMD:C_0805" H 6888 4450 50  0001 C CNN
+F 2 "Capacitors_SMD:C_0805_HandSoldering" H 6888 4450 50  0001 C CNN
 F 3 "" H 6850 4600 50  0000 C CNN
 	1    6850 4600
@@
 	6850 4750 7550 4750
 $Comp
-L GND #PWR705
+L GND #PWR048
 U 1 1 57E4C1C1
 P 7100 4750
-F 0 "#PWR705" H 7100 4500 50  0001 C CNN
+F 0 "#PWR048" H 7100 4500 50  0001 C CNN
 F 1 "GND" H 7100 4600 50  0000 C CNN
 F 2 "" H 7100 4750 50  0000 C CNN
@@
 RX_Q
 $Comp
-L GND #PWR703
+L GND #PWR049
 U 1 1 57E4C1DF
 P 5000 5200
-F 0 "#PWR703" H 5000 4950 50  0001 C CNN
+F 0 "#PWR049" H 5000 4950 50  0001 C CNN
 F 1 "GND" H 5000 5050 50  0000 C CNN
 F 2 "" H 5000 5200 50  0000 C CNN
@@
 	8550 4550 8550 4650
 $Comp
-L +Vlogic #PWR707
+L +Vlogic #PWR050
 U 1 1 57E46B0D
 P 8550 4150
-F 0 "#PWR707" H 8550 3950 50  0001 C CNN
+F 0 "#PWR050" H 8550 3950 50  0001 C CNN
 F 1 "+Vlogic" H 8550 4350 50  0000 C CNN
 F 2 "" H 8550 4150 50  0000 C CNN

Commit message: halfway through layout
Parts:
- added R704, R705: 0R, Resistors_SMD:R_0805_HandSoldering, symbol R
Connections:
- net RX_BIAS: now also R705.1; no longer U702.6 (IN2-), U702.7 (OUT2)
- net TX_BIAS: now also R704.1; no longer U702.1 (OUT1), U702.2 (IN1-)
- new net: R704.2, U702.1 (OUT1), U702.2 (IN1-)
- new net: R705.2, U702.6 (IN2-), U702.7 (OUT2)
Changed lines of the file:
@@
 Connection ~ 7100 4750
 Wire Wire Line
-	7550 4200 7550 4550
+	7550 4100 7550 4550
 Wire Wire Line
 	8550 4550 8550 4650
@@
 L +Vlogic #PWR052
 U 1 1 57E46B0D
-P 8550 4150
-F 0 "#PWR052" H 8550 3950 50  0001 C CNN
-F 1 "+Vlogic" H 8550 4350 50  0000 C CNN
-F 2 "" H 8550 4150 50  0000 C CNN
-F 3 "" H 8550 4150 50  0000 C CNN
-	1    8550 4150
+P 8550 4000
+F 0 "#PWR052" H 8550 3800 50  0001 C CNN
+F 1 "+Vlogic" H 8550 4200 50  0000 C CNN
+F 2 "" H 8550 4000 50  0000 C CNN
+F 3 "" H 8550 4000 50  0000 C CNN
+	1    8550 4000
 	1    0    0    -1
 $EndComp
 Wire Wire Line
-	8550 4150 8550 4450
-Text HLabel 8850 4550 2    60   Output ~ 0
+	8550 4000 8550 4450
+Text HLabel 9000 4550 2    60   Output ~ 0
 RX_BIAS
-Text HLabel 8850 4200 2    60   Output ~ 0
+Text HLabel 8850 4100 2    60   Output ~ 0
 TX_BIAS
-Wire Wire Line
-	7550 4200 8850 4200
 Connection ~ 7550 4450
-Wire Wire Line
-	8550 4550 8850 4550
 Wire Wire Line
 	4825 3850 5050 3850
@@
 Wire Wire Line
 	4600 3950 4125 3950
+$Comp
+L R R704
+U 1 1 57F4AD63
+P 8000 4100
+F 0 "R704" V 8080 4100 50  0000 C CNN
+F 1 "0R" V 8000 4100 50  0000 C CNN
+F 2 "Resistors_SMD:R_0805_HandSoldering" V 7930 4100 50  0001 C CNN
+F 3 "" H 8000 4100 50  0000 C CNN
+	1    8000 4100
+	0    1    1    0
+$EndComp
+Wire Wire Line
+	7550 4100 7850 4100
+Wire Wire Line
+	8150 4100 8850 4100
+$Comp
+L R R705
+U 1 1 57F4AF2B
+P 8750 4550
+F 0 "R705" V 8830 4550 50  0000 C CNN
+F 1 "0R" V 8750 4550 50  0000 C CNN
+F 2 "Resistors_SMD:R_0805_HandSoldering" V 8680 4550 50  0001 C CNN
+F 3 "" H 8750 4550 50  0000 C CNN
+	1    8750 4550
+	0    1    1    0
+$EndComp
+Wire Wire Line
+	8550 4550 8600 4550
+Wire Wire Line
+	8900 4550 9000 4550
 $EndSCHEMATC

Commit message: Changed some component values
Parts:
- R701, R702: value 10k -> 0.1pF
- R703: value 10k -> 1k
Changed lines of the file:
@@
 P 4450 4450
 F 0 "R701" V 4530 4450 50  0000 C CNN
-F 1 "10k" V 4450 4450 50  0000 C CNN
+F 1 "0.1pF" V 4450 4450 50  0000 C CNN
 F 2 "Resistors_SMD:R_0805_HandSoldering" V 4380 4450 50  0001 C CNN
 F 3 "" H 4450 4450 50  0000 C CNN
@@
 P 4650 4450
 F 0 "R702" V 4730 4450 50  0000 C CNN
-F 1 "10k" V 4650 4450 50  0000 C CNN
+F 1 "0.1pF" V 4650 4450 50  0000 C CNN
 F 2 "Resistors_SMD:R_0805_HandSoldering" V 4580 4450 50  0001 C CNN
 F 3 "" H 4650 4450 50  0000 C CNN
@@
 P 5000 5000
 F 0 "R703" V 5080 5000 50  0000 C CNN
-F 1 "10k" V 5000 5000 50  0000 C CNN
+F 1 "1k" V 5000 5000 50  0000 C CNN
 F 2 "Resistors_SMD:R_0805_HandSoldering" V 4930 5000 50  0001 C CNN
 F 3 "" H 5000 5000 50  0000 C CNN
